File: MCU_IO.kicad_sch (KiCad schematic)
At the start: 52 parts, among them Q1 IRLML2803, SW1 B3U-1000P, SW2 B3U-1000P, U1 RP235x-B, U2 TPS3435AFACADDFRQ1, U3 MR25H40MDF, Y1 ABM8-272-T3

Commit message: v5.0 Updates
Parts:
- removed R13, R16: 100k, Resistor_SMD:R_0603_1608Metric, symbol Device:R_Small
- removed R149: 10k, Resistor_SMD:R_0603_1608Metric, symbol Device:R_Small
- added C20: 100n, Capacitor_SMD:C_0603_1608Metric, symbol Device:C_Small
- added R6: 10k, Resistor_SMD:R_0603_1608Metric, symbol Device:R_Small
- added U2: APS6404L-3SQRx-SN, Package_SO:SOIC-8_3.9x4.9mm_P1.27mm, symbol Memory_RAM:APS6404L-3SQRx-SN
- C14: renamed from C13; value 10u -> 4u7
- C18: renamed from C17; value 10p -> 15p
- C19: renamed from C18; value 10p -> 15p
- C23: renamed from C82; value 1u -> 100n; footprint Capacitor_SMD:C_0603_1608Metric -> Capacitor_SMD:C_1210_3225Metric
- L1: value 3.3uH -> AOTA-B201610S3R3-101-T; Field6 (none) -> 3.3uH
- R1: value 220R -> 200R
- R14: value 100k -> 0R; MPN C237792 -> C3029194
- R15: value 100k -> 0R; MPN C237792 -> C3029194; now not fitted; now left out of the parts list
- SW1, SW2: value B3U-1000P -> PTS647; footprint Button_Switch_SMD:SW_SPST_B3U-1000P -> Button_Switch_SMD:SW_SPST_PTS647_Sx38; symbol Switch:SW_Omron_B3FS -> Switch:SW_Push
- U1: value RP235x-B -> RP2350-B
- U3: value MR25H40MDF -> W25Q128JVSIQ; Alternate W25Q32JVSNIQ -> (none); FeRAM (Alt) (none) -> CY15B108QN-40SXI; MRAM (Alt) (none) -> MR25H40MDF
- renumbered C19 to C10, C10 to C11, C11 to C12, C12 to C13, C14 to C15, C15 to C16, C16 to C17, C22 to C21, C21 to C22, C81 to C24, C20 to C25, R9 to R10, R10 to R11, R6 to R12, R7 to R13, R5 to R3, R3 to R4, R4 to R5, R11 to R7, R12 to R8, R8 to R9, U2 to U4
Connections:
- net Battery_ALERT is gone; now on net SPI0_MOSI: U1.80 (GPIO3)
- net COIL_EN is gone; now on net SD_CSn: U1.78 (GPIO1)
- net HEATER0_ON is gone; now on net SPI0_MISO: U1.1 (GPIO4)
- net HEATER1_ON is gone; now on net LoRa_RX_EN: U1.2 (GPIO5)
- net RW_EN is gone; now on net 3V3_M_RST: U1.39 (GPIO31)
- net +3V3_M: now also R14.1, C20.1, R6.1, U2.8 (VDD)
- net 3V3_M_RST: no longer U1.54 (GPIO43/ADC3)
- net 3V3_P_EN: now also U1.38 (GPIO30); no longer U1.53 (GPIO42/ADC2)
- net GND: now also C20.2, U2.4 (VSS); no longer R14.2, U4.5 (SET0)
- net GPS_EN: now also U1.36 (GPIO28); no longer U1.47 (GPIO38)
- net I2C0_SCL: now also U1.42 (GPIO33); no longer U1.26 (GPIO25)
- net I2C0_SDA: now also U1.40 (GPIO32); no longer U1.25 (GPIO24)
- net LoRa_BUSY: now also U1.14 (GPIO15); no longer U1.20 (GPIO20)
- net LoRa_CSn: now also U1.16 (GPIO16); no longer U1.42 (GPIO33)
- net LoRa_EN: now also U1.28 (GPIO27); no longer U1.45 (GPIO36)
- net LoRa_INT: now also U1.17 (GPIO17); no longer U1.21 (GPIO21)
- net LoRa_RSTn: now also U1.13 (GPIO14); no longer U1.19 (GPIO19)
- net LoRa_RX_EN: no longer U1.22 (GPIO22)
- net LoRa_TX_EN: now also U1.3 (GPIO6); no longer U1.23 (GPIO23)
- net NEOPIXEL: now also U1.27 (GPIO26); no longer U1.77 (GPIO0)
- net QSPI_CLK: now also U2.6 (SCLK)
- net QSPI_SD0: now also U2.5 (SI/SIO0)
- net QSPI_SD1: now also U2.2 (SO/SIO1)
- net QSPI_SD2: now also U2.3 (SIO2)
- net QSPI_SD3: now also U2.7 (SIO3)
- net SD_CSn: no longer U1.12 (GPIO13)
- net SPI0_CLK: now also U1.79 (GPIO2); no longer U1.43 (GPIO34)
- net SPI0_MISO: no longer U1.40 (GPIO32)
- net SPI0_MOSI: no longer U1.44 (GPIO35)
- net UART1_RX: now also U1.26 (GPIO25); no longer U1.7 (GPIO9)
- net UART1_TX: now also U1.25 (GPIO24); no longer U1.6 (GPIO8)
- net WDT_EN: now also U1.6 (GPIO8); no longer U1.14 (GPIO15)
- net WDT_WDI: now also U1.4 (GPIO7); no longer U1.79 (GPIO2)
- net IMU_EN: now reaches U1.37 (GPIO29)
- net BUS_IO08: now reaches U1.49 (GPIO40/ADC0)
- net 3V3_P_FLT renamed BUS_IO07
- net GPS_FLT renamed BUS_IO09
- removed net HEATER_ENABLE: R14.1, U1.3 (GPIO6)
- net I2C1_SCL renamed BUS_IO01
- net I2C1_SDA renamed BUS_IO02
- net Jetson_EN renamed SET0
- net SET0: now also R14.2, U4.5 (SET0); no longer U1.4 (GPIO7)
- net Jetson_SD_REQ renamed Mag_CSn
- net LoRa_FLT renamed BUS_IO11
- net RESETn renamed RSTn
- net SPI1_CLK renamed RTC_INT
- net SPI1_MISO renamed Mag_INT
- net SPI1_MOSI renamed Mag_EN
- net UART0_RX renamed BUS_IO03
- net UART0_TX renamed BUS_IO04
- new net BUS_IO05: U1.54 (GPIO43/ADC3)
- new net BUS_IO06: U1.53 (GPIO42/ADC2)
- new net BUS_IO10: U1.47 (GPIO38)
- new net BUS_IO12: U1.45 (GPIO36)
- new net BUS_IO13: U1.44 (GPIO35)
- new net BUS_IO14: U1.43 (GPIO34)
- new net GPS_1PPS: U1.21 (GPIO21)
- new net GPS_RSTn: U1.22 (GPIO22)
- new net IMU_CSn: U1.19 (GPIO19)
- new net IMU_INT1: U1.23 (GPIO23)
- new net IMU_INT2: U1.20 (GPIO20)
- new net PSRAM_CS: R6.2, U1.77 (GPIO0), U2.1 (~{CE})
- new net RTC_EN: U1.7 (GPIO9)
- new net SD_EN: U1.12 (GPIO13)
- no-connect marks 10 -> 1
Other:
- note added: "A: Pinout Option F: Output Topology, Startup Delay: Open-Drain, 10s A: Watchdog Time: External Capacitor C: Time Scaling: 1, 8, 16 A: Output Assert Time: External Capacitor"
- note added: "Flash"
- note added: "Make sure C_{CWD} < 200 x C_{CRST} Use C0G / NP0 Caps for timing stability"
- note added: "Microcontroller"
- note added: "PSRAM"
- note added: "Reset"
- note added: "SET0: Connect to 3V3: WD Multiplier: 8x Connect to GND: WD Multiplier: 1x"
- note added: "T_{WDO} = 4.95 * 10^{6} * C_{RST} T_{WDO} = 0.0495s"
- note added: "T_{WD} = 4.95 * 10^{6} * C_{CWD} * SET0 T_{WD} = 3.96s"
- note added: "Watchdog Timer"
- note removed: "Check Xtal Datasheet This value assumes 10pF crystal bulk capacitance"
- moved on the sheet: C1, C10, C11, C12, C13, C14, C15, C16, C17, C18, C19, C2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
