File: LoRa_Power.kicad_sch (KiCad schematic)
At the start: 18 parts, among them U15 TPS7A4501DCQT, U16 ADM1176-1ARMZ-R7, U7 E22-900M30S

Commit message: Added extra decoupling caps to LoRa
Parts:
- added C26, C27: 1u, Capacitor_SMD:C_0603_1608Metric, symbol Device:C_Small
Connections:
- net GND: now also C26.1, C27.1
- net LoRa_VDD: now also C26.2, C27.2

Commit message: Updated version to v2.1
Other:
- company: (none) -> Carnegie Mellon University
- title: (none) -> Argus Mainboard
Changed lines of the file:
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@@
 	(generator_version "8.0")
 	(paper "A4")
+	(title_block
+		(title "Argus Mainboard")
+		(date "2024-11-19")
+		(rev "v2.1")
+		(company "Carnegie Mellon University")
+		(comment 1 "M. Holliday")
+		(comment 2 "N. Khera")
+		(comment 3 "V. Rajesh")
+	)
 	(junction
 		(at 77.47 58.42)
