File: IMU.kicad_sch (KiCad schematic)
At the start: 10 parts, among them U20 BNO086, Y2 32.768kHz

Commit message: v4.0 Updates
Parts:
- removed C78, C79: 100n, Capacitor_SMD:C_0603_1608Metric, symbol Device:C_Small
- removed C80, C81: 22p, Capacitor_SMD:C_0603_1608Metric, symbol Device:C_Small
- removed R146, R147: 10k, Resistor_SMD:R_0603_1608Metric, symbol Device:R_Small
- removed U20: BNO086, Argus-IC:BNO085, symbol Argus-IC:BNO085
- removed Y2: 32.768kHz, Crystal:Crystal_SMD_MicroCrystal_CC7V-T1A-2Pin_3.2x1.5mm, symbol Device:Crystal
- added C76: 100n, Capacitor_SMD:C_0603_1608Metric, symbol Device:C_Small
- added R136: 10k, Resistor_SMD:R_0603_1608Metric, symbol Device:R_Small
- added U18: BMX160, Argus-IC:BMX160, symbol Argus-IC:BMX160
- renumbered C77 to C75
Connections:
- net +3V3_IMU: now also C76.1, U18.12 (CSB), U18.5 (VDDIO), U18.8 (VDD)
- net GND: now also C76.2, R136.2, U18.2 (GND_1), U18.3 (GND_2), U18.6 (GNDIO), U18.7 (GND_3)
- net IMU_SCL: now also U18.13 (SCX)
- net IMU_SDA: now also U18.14 (SDX)
- new net: R136.1, U18.1 (SDO)
Other:
- sheet I2C Protection1 renamed I2C Protection4
- note added: "0x68"
- note added: "I2C ADDR"
- note added: "IMU"
- note removed: "0x4A"
- note removed: "I2C0 ADDR"
- note removed: "IMU datasheet recommends 12.5pF crystal capacitance"
- note removed: "TODO: BNO085/6?"
- moved on the sheet: C75, F3

Commit message: DFM updates
Parts:
- C75, C76: MPN (none) -> C307348
- R136: MPN (none) -> C2479067
- U18: Flight BMX160 -> (none); MPN (none) -> C2655104; Manufacturer_Name Bosch Sensortec -> (none); Manufacturer_Part_Number BMX160 -> (none); Proto BMX160 -> (none)
Changed lines of the file:
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@@
+			)
+		)
+		(property "MPN" "C307348"
+			(at 124.46 111.76 0)
+			(effects
+				(font
+					(size 1.27 1.27)
+				)
+				(hide yes)
 			)
 		)
@@
 			)
 		)
-		(property "Flight" "BMX160"
-			(at 134.62 97.79 0)
-			(effects
-				(font
-					(size 1.27 1.27)
-				)
-				(hide yes)
-			)
-		)
-		(property "Manufacturer_Name" "Bosch Sensortec"
-			(at 161.29 105.41 0)
-			(effects
-				(font
-					(size 1.27 1.27)
-				)
-				(justify left)
-				(hide yes)
-			)
-		)
-		(property "Manufacturer_Part_Number" "BMX160"
-			(at 149.86 91.44 0)
-			(effects
-				(font
-					(size 1.27 1.27)
-				)
-				(hide yes)
-			)
-		)
-		(property "Proto" "BMX160"
+		(property "MPN" "C2655104"
 			(at 134.62 97.79 0)
 			(effects
@@
 			)
 		)
+		(property "MPN" "C307348"
+			(at 172.72 101.6 0)
+			(effects
+				(font
+					(size 1.27 1.27)
+				)
+				(hide yes)
+			)
+		)
 		(pin "2"
 		)
@@
 			(effects
 				(font
+					(size 1.27 1.27)
+				)
+				(hide yes)
+			)
+		)
+		(property "MPN" "C2479067"
+			(at 124.46 97.79 90)
+			(effects
+				(font
