File: IMU.kicad_sch (KiCad schematic)
At the start: 5 parts, among them U18 BMX160

Commit message: v5.0 Updates
Parts:
- removed C75, C76: 100n, Capacitor_SMD:C_0603_1608Metric, symbol Device:C_Small
- removed F3: 250mA, Fuse:Fuse_0603_1608Metric, symbol Device:Fuse_Small
- removed R136: 10k, Resistor_SMD:R_0603_1608Metric, symbol Device:R_Small
- removed U18: BMX160, Argus-IC:BMX160, symbol Argus-IC:BMX160
- added C81, C82, C83, C85, C86: 10u, Capacitor_SMD:C_0805_2012Metric, symbol Device:C_Small
- added C84: 1u, Capacitor_SMD:C_0603_1608Metric, symbol Device:C_Small
- added C87, C88: 100n, Capacitor_SMD:C_0603_1608Metric, symbol Device:C_Small
- added D17, D18: LED_G_0603_LTST-C190GKT, LED_SMD:LED_0603_1608Metric, symbol Device:LED_Small_Filled
- added R157, R158, R159, R169, R170, R171: 0R, Resistor_SMD:R_0603_1608Metric, symbol Device:R_Small
- added R160, R162, R163, R172, R174, R175, R176, R183, R184: 10k, Resistor_SMD:R_0603_1608Metric, symbol Device:R_Small
- added R161, R173: 2k7, Resistor_SMD:R_0603_1608Metric, symbol Device:R_Small
- added U19, U21: TPS22917DBV, Package_TO_SOT_SMD:SOT-23-6, symbol Power_Management:TPS22917DBV
- added U20: MMC5983MA, Package_LGA:LGA-16_3x3mm_P0.5mm, symbol Argus-IC:MMC5983MA
- added U22: ASM330LHHG1TR, Package_LGA:LGA-14_3x2.5mm_P0.5mm_LayoutBorder3x4y, symbol Sensor_Motion:ISM330DHCX
Connections:
- net +3V3_IMU: now also C86.1, C87.1, C88.1, R171.1, R173.2, R174.2, R175.2, R176.2, R184.2, U21.6 (VOUT), U22.5 (VDDIO), U22.8 (VDD)
- net +3V3_P: now also R158.1, R170.1
- net GND: now also C81.2, C82.2, C83.2, C84.2, C85.2, C86.2, C87.2, C88.2, D17.1 (K), D18.1 (K), R160.2, R172.2, U19.2 (GND), U20.11 (GND), U20.9 (GND), U21.2 (GND), U22.2 (SDx), U22.3 (SCx), U22.6 (GND), U22.7 (GND)
- new net: C81.1, R157.2, R158.2, R159.2, U19.1 (VIN)
- new net: D18.2 (A), R173.1
- new net: R184.1, U21.5 (QOD)
- new net: C83.1, U20.10 (CAP)
- new net: R183.1, U19.5 (QOD)
- new net: C85.1, R169.2, R170.2, R171.2, U21.1 (VIN)
- new net: U20.12 (NC), U20.14 (NC), U20.3 (NC), U20.6 (NC), U20.7 (NC), U20.8 (NC)
- new net: D17.2 (A), R161.1
- new net +3V3_M: R157.1, R169.1
- new net +3V3_MAG: C82.1, C84.1, R159.1, R161.2, R162.2, R163.2, R183.2, U19.6 (VOUT), U20.13 (VDDIO), U20.2 (VDD)
- new net IMU_CSn: R174.1, U22.12 (CS)
- new net IMU_EN: R172.1, U21.3 (ON)
- new net IMU_INT1: R175.1, U22.4 (INT1)
- new net IMU_INT2: R176.1, U22.9 (INT2)
- new net IMU_MISO: U22.1 (SDO/SA0)
- new net IMU_MOSI: U22.14 (SDA)
- new net IMU_SCK: U22.13 (SCL)
- new net Mag_CSn: R162.1, U20.4 (CS)
- new net Mag_EN: R160.1, U19.3 (ON)
- new net Mag_INT: R163.1, U20.15 (INT)
- new net Mag_MISO: U20.5 (MISO)
- new net Mag_MOSI: U20.16 (MOSI)
- new net Mag_SCK: U20.1 (SCK)
Other:
- removed sheet I2C Protection4
- added sheet SPI Protection2 (SPI_Protection.kicad_sch)
- added sheet SPI Protection3 (SPI_Protection.kicad_sch)
- note added: "6-DoF IMU (Accelerometer + Gyroscope)"
- note added: "Magnetometer"
- note removed: "I2C0 ADDR 0x68"
- note removed: "IMU"

Commit message: Final v5.0 Release
Parts:
- R160, R163, R172, R175, R176: value 10k -> 100k
Connections:
- net +3V3_IMU: no longer R175.2, R176.2
- net +3V3_MAG: no longer R163.2
- net GND: now also R163.2, R175.1, R176.1
- net IMU_INT1: now also R175.2; no longer R175.1
- net IMU_INT2: now also R176.2; no longer R176.1
Other:
- moved on the sheet: R162, R163, R174, R175
