File: Payload.kicad_sch (KiCad schematic)
At the start: 1 part, among them U11 XTB-40

Commit message: v3 Layout complete
Parts:
- added C69, C71: 10u, Capacitor_SMD:C_0805_2012Metric, symbol Device:C_Small
- added C70: 100n, Capacitor_SMD:C_0603_1608Metric, symbol Device:C_Small
- added R118: 10k, Resistor_SMD:R_0603_1608Metric, symbol Device:R_Small
- added R119: 100k, Resistor_SMD:R_0603_1608Metric, symbol Device:R_Small
- added R120: 82k5, Resistor_SMD:R_0603_1608Metric, symbol Device:R_Small
- added R121, R122: 0R, Resistor_SMD:R_0603_1608Metric, symbol Device:R_Small
- added U17: AP22653A, Argus-IC:DFN-6-1EP_2x2mm_P0.65mm_EP1x1.6mm, symbol Argus-IC:AP22653
- U18: renamed from U11; footprint mainboard:XTB40_payload -> Argus-Connectors:XTB40_payload; symbol mainboard:XTB-40_payload -> Argus-Connectors:XTB-40_payload
Connections:
- net GND: now reaches U18.1
- net GND: now also U18.10, U18.12, U18.13, U18.14, U18.15, U18.16, U18.17, U18.19, U18.2, U18.20, U18.23, U18.3, U18.8, C69.1, C70.1, C71.1, R119.2, R120.2, U17.5 (GND), U17.7 (EP)
- net at U18.11: now also R121.2, R122.2
- net Payload_IO2: now reaches U18.18
- net Payload_IO1: now reaches U18.21
- net Payload_IO0: now reaches U18.22
- net Payload_SCK: now reaches U18.4
- net Payload_MOSI: now reaches U18.5
- net Payload_MISO: now reaches U18.6
- net Payload_CSn: now reaches U18.7
- net VDD_PAYLOAD: now reaches U18.9
- net VDD_PAYLOAD: now also C71.2, R121.1, U17.1 (OUT)
- new net: R120.1, U17.2 (ISET)
- new net +3V3_P: C69.2, C70.2, R118.1, U17.6 (IN)
- new net Payload_EN: R119.1, U17.4 (EN)
- new net Payload_FLT: R118.2, U17.3 (FLG)
- new net VSYS: R122.1
Other:
- added sheet SPI Protection2 (SPI_Protection.kicad_sch)
- note added: "ILimit_Min = 28955 / R^1.075 = 0.150 mA Ilimit_Typ = 30321 / R^1.055 = 0.197 mA ILimit_Max = 31033 / R^1.031 = 0.264 mA"

Commit message: Addressed design issues
Parts:
- R121: now fitted
Connections:
- net +3V3_P: no longer R118.1
- new net +3V3_M: R118.1
Other:
- note added: "ILimit_Min = 28955 / R^1.075 = 0.150 A Ilimit_Typ = 30321 / R^1.055 = 0.197 A ILimit_Max = 31033 / R^1.031 = 0.264 A"
- note removed: "ILimit_Min = 28955 / R^1.075 = 0.150 mA Ilimit_Typ = 30321 / R^1.055 = 0.197 mA ILimit_Max = 31033 / R^1.031 = 0.264 mA"
Changed lines of the file:
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@@
-	)
-	(junction
-		(at 97.79 59.69)
-		(diameter 0)
-		(color 0 0 0 0)
 	)
 	(junction
@@
 	(wire
 		(pts
+			(xy 97.79 58.42) (xy 97.79 60.96)
+		)
+		(stroke
+			(width 0)
+			(type default)
+		)
+	)
+	(wire
+		(pts
 			(xy 121.92 119.38) (xy 125.73 119.38)
 		)
@@
 	(wire
 		(pts
-			(xy 77.47 59.69) (xy 97.79 59.69)
-		)
-		(stroke
-			(width 0)
-			(type default)
-		)
-	)
-	(wire
-		(pts
 			(xy 116.84 72.39) (xy 118.11 72.39)
 		)
@@
 	(wire
 		(pts
-			(xy 97.79 59.69) (xy 97.79 60.96)
-		)
-		(stroke
-			(width 0)
-			(type default)
-		)
-	)
-	(wire
-		(pts
 			(xy 226.06 63.5) (xy 247.65 63.5)
 		)
@@
 	(wire
 		(pts
-			(xy 97.79 59.69) (xy 101.6 59.69)
+			(xy 77.47 59.69) (xy 101.6 59.69)
 		)
 		(stroke
@@
 		)
 	)
-	(text "ILimit_Min = 28955 / R^1.075 = 0.150 mA\nIlimit_Typ = 30321 / R^1.055 = 0.197 mA\nILimit_Max = 31033 / R^1.031 = 0.264 mA"
+	(text "ILimit_Min = 28955 / R^1.075 = 0.150 A\nIlimit_Typ = 30321 / R^1.055 = 0.197 A\nILimit_Max = 31033 / R^1.031 = 0.264 A"
 		(exclude_from_sim no)
 		(at 136.652 89.154 0)
@@
 				(path "/4c932743-8c6f-426e-9c1f-5a3f2b32c70d/0c04e6a7-6d16-45e0-b82f-bf6f349905a8"
 					(reference "#PWR026")
+					(unit 1)
+				)
+			)
+		)
+	)
+	(symbol
+		(lib_id "power:+3.3V")
+		(at 97.79 58.42 0)
+		(unit 1)
+		(exclude_from_sim no)
+		(in_bom yes)
+		(on_board yes)
+		(dnp no)
+		(property "Reference" "#SUPPLY8"
+			(at 97.79 58.42 0)
+			(effects
+				(font
+					(size 1.27 1.27)
+				)
+				(hide yes)
+			)
+		)
+		(property "Value" "+3V3_M"
+			(at 97.79 54.61 0)
+			(effects
+				(font
+					(size 1.27 1.27)
+				)
+			)
+		)
+		(property "Footprint" ""
+			(at 97.79 58.42 0)
+			(effects
+				(font
+					(size 1.27 1.27)
+				)
+				(hide yes)
+			)
+		)
+		(property "Datasheet" ""
+			(at 97.79 58.42 0)
+			(effects
+				(font
+					(size 1.27 1.27)
+				)
+				(hide yes)
+			)
+		)
+		(property "Description" "Power symbol creates a global label with name \"+3.3V\""
+			(at 97.79 58.42 0)
+			(effects
+				(font
+					(size 1.27 1.27)
+				)
+				(hide yes)
+			)
+		)
+		(pin "1"
+		)
+		(instances
+			(project "Avionics-MainBoard"
+				(path "/4c932743-8c6f-426e-9c1f-5a3f2b32c70d/0c04e6a7-6d16-45e0-b82f-bf6f349905a8"
+					(reference "#SUPPLY8")
 					(unit 1)
 				)
@@
 		(in_bom yes)
 		(on_board yes)
-		(dnp yes)
+		(dnp no)
 		(property "Reference" "R121"
 			(at 135.89 141.224 0)
