File: GPS.kicad_sch (KiCad schematic)
At the start: 18 parts, among them J7 U.FL-R-SMT-1, Q2 IRLML2803, Q6 IRF7404, U10 AP22653A, U8 S1216V8

Commit message: v3 partial schematic updates
Parts:
- F2: symbol Device:Polyfuse_Small -> Device:Fuse_Small
Connections:
- net +3V3_P: now also F2.2; no longer F2.1
- net at Q6.1 (Source), Q6.2 (Source), Q6.3 (Source)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: now also F2.1; no longer F2.2
Other:
- note added: "GPS Enable"
- note added: "GPS Module"
- note removed: "GPS Power"
Changed lines of the file:
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@@
 		)
 	)
-	(text "GPS Power"
+	(text "GPS Enable"
 		(exclude_from_sim no)
 		(at 81.026 47.498 0)
@@
 			)
 			(justify left bottom)
+		)
+	)
+	(text "GPS Module"
+		(exclude_from_sim no)
+		(at 191.77 67.31 0)
+		(effects
+			(font
+				(size 2.54 2.54)
+			)
+			(justify bottom)
 		)
 	)
@@
 		)
 		(instances
-			(project ""
+			(project "Avionics-MainBoard"
 				(path "/4c932743-8c6f-426e-9c1f-5a3f2b32c70d/1ff82478-f00f-4d48-a429-2ed9117c0498"
 					(reference "U8")
@@
 	)
 	(symbol
-		(lib_id "Device:Polyfuse_Small")
-		(at 73.66 60.96 0)
+		(lib_id "Device:Fuse_Small")
+		(at 73.66 60.96 90)
 		(unit 1)
 		(exclude_from_sim no)
@@
 		(dnp no)
 		(property "Reference" "F2"
-			(at 72.39 59.944 0)
+			(at 69.342 59.944 90)
 			(effects
 				(font
@@
 		)
 		(property "Value" "250mA"
-			(at 72.39 61.976 0)
+			(at 65.278 61.976 90)
 			(effects
 				(font
@@
 		)
 		(property "Footprint" ""
-			(at 74.93 66.04 0)
-			(effects
-				(font
-					(size 1.27 1.27)
-				)
-				(justify left)
+			(at 73.66 60.96 0)
+			(effects
+				(font
+					(size 1.27 1.27)
+				)
 				(hide yes)
 			)
@@
 			)
 		)
-		(property "Description" "Resettable fuse, polymeric positive temperature coefficient, small symbol"
+		(property "Description" "Fuse, small symbol"
 			(at 73.66 60.96 0)
 			(effects
@@
 		)
 		(instances
-			(project ""
+			(project "Avionics-MainBoard"
 				(path "/4c932743-8c6f-426e-9c1f-5a3f2b32c70d/1ff82478-f00f-4d48-a429-2ed9117c0498"
 					(reference "F2")

Commit message: v3 Layout complete
Parts:
- removed F2: 250mA, symbol Device:Fuse_Small
- removed Q2: IRLML2803, Package_TO_SOT_SMD:SOT-23, symbol Mainboard:IRLML2803
- removed Q6: IRF7404, Package_SO:SOIC-8_3.9x4.9mm_P1.27mm, symbol Mainboard:IRF7404
- removed R30: 10k, Resistor_SMD:R_0603_1608Metric, symbol Device:R_Small
- removed R31: 4k7, Resistor_SMD:R_0603_1608Metric, symbol Device:R_Small
- removed R32: 3k3, Resistor_SMD:R_0603_1608Metric, symbol Device:R_Small
- added C88: 1u, Capacitor_SMD:C_0603_1608Metric, symbol Device:C_Small
- C66: renamed from C16; footprint Capacitor_SMD:C_0603_1608Metric -> Capacitor_SMD:C_0805_2012Metric
- C68: renamed from C25; footprint Capacitor_SMD:C_0603_1608Metric -> Capacitor_SMD:C_0805_2012Metric
- U15: renamed from U10; footprint JetsonCarrier:DFN-6-1EP_2x2mm_P0.65mm_EP1x1.6mm -> Argus-IC:DFN-6-1EP_2x2mm_P0.65mm_EP1x1.6mm; symbol JetsonCarrier:AP22653 -> Argus-IC:AP22653
- U16: renamed from U8; value S1216V8 -> PX1120S
- renumbered C15 to C67, J7 to J3, R36 to R112, R37 to R113, R38 to R114, R10 to R115, R11 to R116, R12 to R117
Connections:
- net GND: now also C88.1
- net VDD_GPS: now also C88.2
Other:
- note removed: "TODO: Pick one"
- moved on the sheet: C66, C67, C68, J3, R112, R113, R114, R115, R116, R117, U15, U16

Commit message: Addressed design issues
Parts:
- R114: value 82k5 -> 49k9
Connections:
- net +3V3_P: no longer R112.1
- new net +3V3_M: R112.1
Other:
- note added: "ILimit_Min = 28955 / R^1.075 = 0.441 A Ilimit_Typ = 30321 / R^1.055 = 0.490 A ILimit_Max = 31033 / R^1.031 = 0.539 A"
- note removed: "ILimit_Min = 28955 / R^1.075 = 0.150 mA Ilimit_Typ = 30321 / R^1.055 = 0.197 mA ILimit_Max = 31033 / R^1.031 = 0.264 mA"
- moved on the sheet: R114
Changed lines of the file:
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@@
-	)
-	(junction
-		(at 77.47 93.98)
-		(diameter 0)
-		(color 0 0 0 0)
 	)
 	(junction
@@
 	(wire
 		(pts
-			(xy 77.47 93.98) (xy 77.47 95.25)
-		)
-		(stroke
-			(width 0)
-			(type default)
-		)
-	)
-	(wire
-		(pts
 			(xy 182.88 116.84) (xy 177.8 116.84)
 		)
@@
 	(wire
 		(pts
+			(xy 77.47 92.71) (xy 77.47 95.25)
+		)
+		(stroke
+			(width 0)
+			(type default)
+		)
+	)
+	(wire
+		(pts
 			(xy 218.44 88.9) (xy 242.57 88.9)
 		)
@@
 	(wire
 		(pts
-			(xy 104.14 101.6) (xy 104.14 105.41)
+			(xy 102.87 101.6) (xy 102.87 105.41)
 		)
 		(stroke
@@
 	(wire
 		(pts
-			(xy 77.47 93.98) (xy 81.28 93.98)
-		)
-		(stroke
-			(width 0)
-			(type default)
-		)
-	)
-	(wire
-		(pts
-			(xy 96.52 101.6) (xy 104.14 101.6)
+			(xy 96.52 101.6) (xy 102.87 101.6)
 		)
 		(stroke
@@
 	(wire
 		(pts
-			(xy 62.23 93.98) (xy 77.47 93.98)
+			(xy 62.23 93.98) (xy 81.28 93.98)
 		)
 		(stroke
@@
 	(wire
 		(pts
-			(xy 104.14 113.03) (xy 104.14 110.49)
+			(xy 102.87 113.03) (xy 102.87 110.49)
 		)
 		(stroke
@@
 		)
 	)
-	(text "ILimit_Min = 28955 / R^1.075 = 0.150 mA\nIlimit_Typ = 30321 / R^1.055 = 0.197 mA\nILimit_Max = 31033 / R^1.031 = 0.264 mA"
+	(text "ILimit_Min = 28955 / R^1.075 = 0.441 A\nIlimit_Typ = 30321 / R^1.055 = 0.490 A\nILimit_Max = 31033 / R^1.031 = 0.539 A"
 		(exclude_from_sim no)
 		(at 116.332 123.444 0)
@@
 	(symbol
 		(lib_id "power:GND")
-		(at 104.14 113.03 0)
+		(at 102.87 113.03 0)
 		(unit 1)
 		(exclude_from_sim no)
@@
 		(dnp no)
 		(property "Reference" "#PWR058"
-			(at 104.14 119.38 0)
+			(at 102.87 119.38 0)
 			(effects
 				(font
@@
 		)
 		(property "Value" "GND"
-			(at 102.235 116.84 0)
+			(at 100.965 116.84 0)
 			(effects
 				(font
@@
 		)
 		(property "Footprint" ""
-			(at 104.14 113.03 0)
+			(at 102.87 113.03 0)
 			(effects
 				(font
@@
 		)
 		(property "Datasheet" ""
-			(at 104.14 113.03 0)
+			(at 102.87 113.03 0)
 			(effects
 				(font
@@
 		)
 		(property "Description" "Power symbol creates a global label with name \"GND\" , ground"
-			(at 104.14 113.03 0)
+			(at 102.87 113.03 0)
 			(effects
 				(font
@@
 		)
 		(property "Author" "Antmicro"
-			(at 113.03 120.65 0)
+			(at 111.76 120.65 0)
 			(effects
 				(font
@@
 		)
 		(property "License" "Apache-2.0"
-			(at 113.03 123.19 0)
+			(at 111.76 123.19 0)
 			(effects
 				(font
@@
 	)
 	(symbol
+		(lib_id "power:+3.3V")
+		(at 77.47 92.71 0)
+		(unit 1)
+		(exclude_from_sim no)
+		(in_bom yes)
+		(on_board yes)
+		(dnp no)
+		(property "Reference" "#SUPPLY3"
+			(at 77.47 92.71 0)
+			(effects
+				(font
+					(size 1.27 1.27)
+				)
+				(hide yes)
+			)
+		)
+		(property "Value" "+3V3_M"
+			(at 77.47 88.9 0)
+			(effects
+				(font
+					(size 1.27 1.27)
+				)
+			)
+		)
+		(property "Footprint" ""
+			(at 77.47 92.71 0)
+			(effects
+				(font
+					(size 1.27 1.27)
+				)
+				(hide yes)
+			)
+		)
+		(property "Datasheet" ""
+			(at 77.47 92.71 0)
+			(effects
+				(font
+					(size 1.27 1.27)
+				)
+				(hide yes)
+			)
+		)
+		(property "Description" "Power symbol creates a global label with name \"+3.3V\""
+			(at 77.47 92.71 0)
+			(effects
+				(font
+					(size 1.27 1.27)
+				)
+				(hide yes)
+			)
+		)
+		(pin "1"
+		)
+		(instances
+			(project "Avionics-MainBoard"
+				(path "/4c932743-8c6f-426e-9c1f-5a3f2b32c70d/1ff82478-f00f-4d48-a429-2ed9117c0498"
+					(reference "#SUPPLY3")
+					(unit 1)
+				)
+			)
+		)
+	)
+	(symbol
 		(lib_id "Device:C_Small")
 		(at 173.99 118.11 0)
@@
 	(symbol
 		(lib_id "Device:R_Small")
-		(at 104.14 107.95 0)
+		(at 102.87 107.95 0)
 		(unit 1)
 		(exclude_from_sim no)
@@
 		(dnp no)
 		(property "Reference" "R114"
-			(at 105.41 106.934 0)
+			(at 104.14 106.934 0)
 			(effects
 				(font
@@
 			)
 		)
-		(property "Value" "82k5"
-			(at 105.41 109.728 0)
+		(property "Value" "49k9"
+			(at 104.14 109.728 0)
 			(effects
 				(font
@@
 		)
 		(property "Footprint" "Resistor_SMD:R_0603_1608Metric"
-			(at 104.14 107.95 0)
+			(at 102.87 107.95 0)
 			(effects
 				(font
@@
 		)
 		(property "Datasheet" "~"
-			(at 104.14 107.95 0)
+			(at 102.87 107.95 0)
 			(effects
 				(font
@@
 		)
 		(property "Description" "Resistor, small symbol"
-			(at 104.14 107.95 0)
+			(at 102.87 107.95 0)
 			(effects
 				(font
@@
 		)
 		(property "Manufacturer" "Bourns"
-			(at 124.46 130.81 0)
+			(at 123.19 130.81 0)
 			(effects
 				(font
@@
 		)
 		(property "MPN" "CR0402-FX-1502GLF"
-			(at 124.46 128.27 0)
+			(at 123.19 128.27 0)
 			(effects
 				(font
@@
 		)
 		(property "Val" "15k"
-			(at 105.41 109.22 90)
+			(at 104.14 109.22 90)
 			(effects
 				(font
@@
 		)
 		(property "License" "Apache-2.0"
-			(at 124.46 133.35 0)
+			(at 123.19 133.35 0)
 			(effects
 				(font
@@
 		)
 		(property "Author" "Antmicro"
-			(at 124.46 135.89 0)
+			(at 123.19 135.89 0)
 			(effects
 				(font
@@
 		)
 		(property "Tolerance" "1%"
-			(at 124.46 118.11 0)
-			(effects
-				(font
+			(at 123.19 118.11 0)
+			(effects
+				(font

Commit message: v4.0 Updates
Parts:
- renumbered C88 to C69

Commit message: DFM updates
Parts:
- C66, C68: Author Antmicro -> (none); Dielectric X5R -> (none); License Apache-2.0 -> (none); MPN GRM155R61H104KE14D -> C386084; Manufacturer Murata -> (none); Val 100n -> (none); Voltage 50V -> (none)
- C67: Author Antmicro -> (none); Dielectric X5R -> (none); License Apache-2.0 -> (none); MPN GRM155R61H104KE14D -> C307348; Manufacturer Murata -> (none); Val 100n -> (none); Voltage 50V -> (none)
- C69: Author Antmicro -> (none); Dielectric X5R -> (none); License Apache-2.0 -> (none); MPN GRM155R61H104KE14D -> C2214844; Manufacturer Murata -> (none); Val 100n -> (none); Voltage 50V -> (none)
- J3: MPN (none) -> C88374
- R112: Author Antmicro -> (none); License Apache-2.0 -> (none); MPN CR0402-FX-1003GLF -> C2479067; Manufacturer Bourns -> (none); Tolerance 1% -> (none); Val 100k -> (none)
- R113: Author Antmicro -> (none); License Apache-2.0 -> (none); MPN CR0402-FX-1003GLF -> C237792; Manufacturer Bourns -> (none); Tolerance 1% -> (none); Val 100k -> (none)
- R114: Author Antmicro -> (none); License Apache-2.0 -> (none); MPN CR0402-FX-1502GLF -> C844789; Manufacturer Bourns -> (none); Tolerance 1% -> (none); Val 15k -> (none)
- R115, R116: MPN (none) -> C844915
- R117: MPN (none) -> C2479067
- U15: Author Antmicro -> (none); License Apache-2.0 -> (none); MPN AP22653FDZ-7 -> C1511768; Manufacturer Diodes Incorporated -> (none)

Commit message: v4.2 Updates
Parts:
- added R151, R152: 0R, Resistor_SMD:R_0603_1608Metric, symbol Device:R_Small
Connections:
- net +3V3_M: now also R152.1
- net +3V3_P: now also R151.1; no longer C66.2, C67.2, U15.6 (IN)
- new net: C66.2, C67.2, R151.2, R152.2, U15.6 (IN)
Changed lines of the file:
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@@
 	(title_block
 		(title "Argus Mainboard")
-		(date "2025-01-08")
-		(rev "v3.0")
+		(date "2025-11-24")
+		(rev "v4.2")
 		(company "Carnegie Mellon University")
 		(comment 1 "M. Holliday")
@@
 	(wire
 		(pts
+			(xy 62.23 91.44) (xy 62.23 93.98)
+		)
+		(stroke
+			(width 0)
+			(type default)
+		)
+	)
+	(wire
+		(pts
 			(xy 177.8 111.76) (xy 177.8 114.3)
 		)
@@
 	(wire
 		(pts
+			(xy 62.23 83.82) (xy 62.23 86.36)
+		)
+		(stroke
+			(width 0)
+			(type default)
+		)
+	)
+	(wire
+		(pts
 			(xy 96.52 106.68) (xy 97.79 106.68)
 		)
@@
 	(wire
 		(pts
-			(xy 53.34 92.71) (xy 53.34 93.98)
+			(xy 53.34 83.82) (xy 53.34 86.36)
 		)
 		(stroke
@@
 		(pts
 			(xy 53.34 100.33) (xy 53.34 101.6)
+		)
+		(stroke
+			(width 0)
+			(type default)
+		)
+	)
+	(wire
+		(pts
+			(xy 53.34 91.44) (xy 53.34 93.98)
 		)
 		(stroke
@@
 	)
 	(symbol
+		(lib_id "Device:R_Small")
+		(at 53.34 88.9 0)
+		(unit 1)
+		(exclude_from_sim no)
+		(in_bom yes)
+		(on_board yes)
+		(dnp no)
+		(property "Reference" "R151"
+			(at 52.07 87.884 0)
+			(effects
+				(font
+					(size 1.27 1.27)
+				)
+				(justify right)
+			)
+		)
+		(property "Value" "0R"
+			(at 52.07 89.916 0)
+			(effects
+				(font
+					(size 1.27 1.27)
+				)
+				(justify right)
+			)
+		)
+		(property "Footprint" "Resistor_SMD:R_0603_1608Metric"
+			(at 53.34 88.9 0)
+			(effects
+				(font
+					(size 1.27 1.27)
+				)
+				(hide yes)
+			)
+		)
+		(property "Datasheet" "~"
+			(at 53.34 88.9 0)
+			(effects
+				(font
+					(size 1.27 1.27)
+				)
+				(hide yes)
+			)
+		)
+		(property "Description" "Resistor, small symbol"
+			(at 53.34 88.9 0)
+			(effects
+				(font
+					(size 1.27 1.27)
+				)
+				(hide yes)
+			)
+		)
+		(pin "1"
+		)
+		(pin "2"
+		)
+		(instances
+			(project ""
+				(path "/4c932743-8c6f-426e-9c1f-5a3f2b32c70d/1ff82478-f00f-4d48-a429-2ed9117c0498"
+					(reference "R151")
+					(unit 1)
+				)
+			)
+		)
+	)
+	(symbol
 		(lib_id "Argus-IC:AP22653")
 		(at 81.28 99.06 0)
@@
 	(symbol
 		(lib_id "power:+3.3V")
+		(at 62.23 83.82 0)
+		(unit 1)
+		(exclude_from_sim no)
+		(in_bom yes)
+		(on_board yes)
+		(dnp no)
+		(property "Reference" "#SUPPLY08"
+			(at 62.23 83.82 0)
+			(effects
+				(font
+					(size 1.27 1.27)
+				)
+				(hide yes)
+			)
+		)
+		(property "Value" "+3V3_M"
+			(at 62.23 80.01 0)
+			(effects
+				(font
+					(size 1.27 1.27)
+				)
+			)
+		)
+		(property "Footprint" ""
+			(at 62.23 83.82 0)
+			(effects
+				(font
+					(size 1.27 1.27)
+				)
+				(hide yes)
+			)
+		)
+		(property "Datasheet" ""
+			(at 62.23 83.82 0)
+			(effects
+				(font
+					(size 1.27 1.27)
+				)
+				(hide yes)
+			)
+		)
+		(property "Description" "Power symbol creates a global label with name \"+3.3V\""
+			(at 62.23 83.82 0)
+			(effects
+				(font
+					(size 1.27 1.27)
+				)
+				(hide yes)
+			)
+		)
+		(pin "1"
+		)
+		(instances
+			(project "Avionics-MainBoard"
+				(path "/4c932743-8c6f-426e-9c1f-5a3f2b32c70d/1ff82478-f00f-4d48-a429-2ed9117c0498"
+					(reference "#SUPPLY08")
+					(unit 1)
+				)
+			)
+		)
+	)
+	(symbol
+		(lib_id "power:+3.3V")
 		(at 111.76 92.71 0)
 		(unit 1)
@@
 	(symbol
 		(lib_id "power:+3.3V")
-		(at 53.34 92.71 0)
+		(at 53.34 83.82 0)
 		(unit 1)
 		(exclude_from_sim no)
@@
 		(dnp no)
 		(property "Reference" "#SUPPLY018"
-			(at 53.34 92.71 0)
+			(at 53.34 83.82 0)
 			(effects
 				(font
@@
 		)
 		(property "Value" "+3V3_P"
-			(at 53.34 88.9 0)
+			(at 53.34 80.01 0)
 			(effects
 				(font
@@
 		)
 		(property "Footprint" ""
-			(at 53.34 92.71 0)
+			(at 53.34 83.82 0)
 			(effects
 				(font
@@
 		)
 		(property "Datasheet" ""
-			(at 53.34 92.71 0)
+			(at 53.34 83.82 0)
 			(effects
 				(font
@@
 		)
 		(property "Description" "Power symbol creates a global label with name \"+3.3V\""
-			(at 53.34 92.71 0)
+			(at 53.34 83.82 0)
 			(effects
 				(font
@@
 					(unit 1)
 				)
+			)
+		)
+	)
+	(symbol
+		(lib_id "Device:R_Small")
+		(at 62.23 88.9 0)
+		(unit 1)
+		(exclude_from_sim no)
+		(in_bom yes)
+		(on_board yes)
+		(dnp yes)
+		(property "Reference" "R152"
+			(at 60.96 87.884 0)
+			(effects
+				(font
+					(size 1.27 1.27)
+				)
+				(justify right)
+			)
+		)
+		(property "Value" "0R"
+			(at 60.96 89.916 0)
+			(effects
+				(font
+					(size 1.27 1.27)
+				)
+				(justify right)
+			)
+		)
+		(property "Footprint" "Resistor_SMD:R_0603_1608Metric"
+			(at 62.23 88.9 0)
+			(effects
+				(font
+					(size 1.27 1.27)
+				)
+				(hide yes)
+			)
+		)
+		(property "Datasheet" "~"
+			(at 62.23 88.9 0)
+			(effects
+				(font
+					(size 1.27 1.27)
+				)
+				(hide yes)
+			)
+		)
+		(property "Description" "Resistor, small symbol"
+			(at 62.23 88.9 0)
+			(effects
+				(font
+					(size 1.27 1.27)
+				)
+				(hide yes)
+			)
+		)
+		(pin "1"
+		)
+		(pin "2"
+		)
+		(instances
+			(project "Avionics-MainBoard"
+				(path "/4c932743-8c6f-426e-9c1f-5a3f2b32c70d/1ff82478-f00f-4d48-a429-2ed9117c0498"
+					(reference "R152")
+					(unit 1)
+				)
