File: GPS.kicad_sch (KiCad schematic)
At the start: 15 parts, among them J3 U.FL-R-SMT-1, U15 AP22653A, U16 PX1120S

Commit message: v5.0 Updates
Parts:
- removed C69: 1u, Capacitor_SMD:C_0603_1608Metric, symbol Device:C_Small
- added BT1: MS621FE-FL11E, Battery:BatteryHolder_Seiko_MS621F, symbol Device:Battery_Cell
- added C68: 1u, Capacitor_SMD:C_0603_1608Metric, symbol Device:C_Small
- added D13: LED_G_0603_LTST-C190GKT, LED_SMD:LED_0603_1608Metric, symbol Device:LED_Small_Filled
- added D14: DFLS130LQ-7, Diode_SMD:D_PowerDI-123, symbol Device:D_Schottky
- added R121: 2k7, Resistor_SMD:R_0603_1608Metric, symbol Device:R_Small
- added R124: 1k, Resistor_SMD:R_0603_1608Metric, symbol Device:R_Small
- added R125: 10k, Resistor_SMD:R_0603_1608Metric, symbol Device:R_Small
- added TP3: TestPoint, TestPoint:TestPoint_Pad_D1.5mm, symbol Connector:TestPoint
- J12: renamed from J3; value U.FL-R-SMT-1 -> 60612202111308; footprint Connector_Coaxial:U.FL_Hirose_U.FL-R-SMT-1_Vertical -> Argus-Connectors:60612202111308
- R117: value 10k -> 0R; now not fitted; now left out of the parts list
- renumbered C66 to C65, C67 to C66, C68 to C67, R151 to R115, R152 to R116, R112 to R118, R113 to R119, R114 to R120, R115 to R122, R116 to R123, U15 to U14, U16 to U15
Connections:
- net GND: now also BT1.2 (-), C68.1, D13.1 (K)
- net VDD_GPS: now also R117.1, D14.2 (A), R121.2, R125.1; no longer R117.2, U15.22 (V_BCKP)
- net at C65.2, C66.2, R115.2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: now also R117.2
- net GPS_RSTn: now reaches U15.8 (RSTN)
- net GPS_RSTn: now also R125.2; no longer R117.1
- net GPS_1PPS: now reaches U15.3 (1PPS)
- net GPS_FLT: no longer names the net of R118.2, U14.3 (FLG)
- net GPS_FLT: now also TP3.1
- new net: BT1.1 (+), C68.2, R124.1, U15.22 (V_BCKP)
- new net: D14.1 (K), R124.2
- new net: D13.2 (A), R121.1
- no-connect marks 14 -> 13
Other:
- note added: "ILimit_Min = 28955 / R[kOhm]^1.075 = 441mA = 0.441 A Ilimit_Typ = 30321 / R[kOhm]^1.055 = 490mA = 0.490 A ILimit_Max = 31033 / R[kOhm]^1.031 = 539mA = 0.539 A"
- note removed: "ILimit_Min = 28955 / R^1.075 = 0.441 A Ilimit_Typ = 30321 / R^1.055 = 0.490 A ILimit_Max = 31033 / R^1.031 = 0.539 A"
- moved on the sheet: C65, C66, C67, J12, R115, R116, R118, R119, R120, R122, R123, U14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

Commit message: Final v5.0 Release
Parts:
- removed D14: DFLS130LQ-7, Diode_SMD:D_PowerDI-123, symbol Device:D_Schottky
- added D14: BAT54W, Package_TO_SOT_SMD:SOT-323_SC-70, symbol Diode:BAT54W
- added R186: 0R, Resistor_SMD:R_0603_1608Metric, symbol Device:R_Small
Connections:
- net GPS_1PPS: now also R186.2; no longer U15.3 (1PPS)
- net VDD_GPS: now also D14.1 (A)
- net at R124.2: now also D14.3 (K)
- new net: R186.1, U15.3 (1PPS)
Changed lines of the file:
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@@
 	(wire
 		(pts
+			(xy 229.235 111.76) (xy 226.06 111.76)
+		)
+		(stroke
+			(width 0)
+			(type default)
+		)
+	)
+	(wire
+		(pts
 			(xy 66.675 107.315) (xy 68.58 107.315)
 		)
@@
 	(wire
 		(pts
+			(xy 237.49 111.76) (xy 234.315 111.76)
+		)
+		(stroke
+			(width 0)
+			(type default)
+		)
+	)
+	(wire
+		(pts
 			(xy 162.56 111.76) (xy 167.64 111.76)
 		)
@@
 	(hierarchical_label "GPS_1PPS"
 		(shape output)
-		(at 226.06 111.76 0)
+		(at 237.49 111.76 0)
 		(effects
 			(font
@@
 	)
 	(symbol
+		(lib_id "Diode:BAT54W")
+		(at 149.86 111.76 180)
+		(unit 1)
+		(body_style 1)
+		(exclude_from_sim no)
+		(in_bom yes)
+		(on_board yes)
+		(in_pos_files yes)
+		(dnp no)
+		(property "Reference" "D14"
+			(at 149.86 114.3 0)
+			(show_name no)
+			(do_not_autoplace no)
+			(effects
+				(font
+					(size 1.27 1.27)
+				)
+			)
+		)
+		(property "Value" "BAT54W"
+			(at 149.86 116.205 0)
+			(show_name no)
+			(do_not_autoplace no)
+			(effects
+				(font
+					(size 1.27 1.27)
+				)
+			)
+		)
+		(property "Footprint" "Package_TO_SOT_SMD:SOT-323_SC-70"
+			(at 149.86 107.315 0)
+			(hide yes)
+			(show_name no)
+			(do_not_autoplace no)
+			(effects
+				(font
+					(size 1.27 1.27)
+				)
+			)
+		)
+		(property "Datasheet" "https://assets.nexperia.com/documents/data-sheet/BAT54W_SER.pdf"
+			(at 149.86 111.76 0)
+			(hide yes)
+			(show_name no)
+			(do_not_autoplace no)
+			(effects
+				(font
+					(size 1.27 1.27)
+				)
+			)
+		)
+		(property "Description" "Schottky barrier diode, SOT-323"
+			(at 149.86 111.76 0)
+			(hide yes)
+			(show_name no)
+			(do_not_autoplace no)
+			(effects
+				(font
+					(size 1.27 1.27)
+				)
+			)
+		)
+		(pin "1"
+		)
+		(pin "3"
+		)
+		(pin "2"
+		)
+		(instances
+			(project "Avionics-MainBoard"
+				(path "/4c932743-8c6f-426e-9c1f-5a3f2b32c70d/1ff82478-f00f-4d48-a429-2ed9117c0498"
+					(reference "D14")
+					(unit 1)
+				)
+			)
+		)
+	)
+	(symbol
 		(lib_id "power:GND")
 		(at 113.665 116.205 0)
@@
 	)
 	(symbol
+		(lib_id "Device:R_Small")
+		(at 231.775 111.76 90)
+		(unit 1)
+		(body_style 1)
+		(exclude_from_sim no)
+		(in_bom yes)
+		(on_board yes)
+		(in_pos_files yes)
+		(dnp no)
+		(property "Reference" "R186"
+			(at 231.775 107.95 90)
+			(show_name no)
+			(do_not_autoplace no)
+			(effects
+				(font
+					(size 1.27 1.27)
+				)
+			)
+		)
+		(property "Value" "0R"
+			(at 231.775 109.855 90)
+			(show_name no)
+			(do_not_autoplace no)
+			(effects
+				(font
+					(size 1.27 1.27)
+				)
+			)
+		)
+		(property "Footprint" "Resistor_SMD:R_0603_1608Metric"
+			(at 231.775 111.76 0)
+			(hide yes)
+			(show_name no)
+			(do_not_autoplace no)
+			(effects
+				(font
+					(size 1.27 1.27)
+				)
+			)
+		)
+		(property "Datasheet" ""
+			(at 231.775 111.76 0)
+			(hide yes)
+			(show_name no)
+			(do_not_autoplace no)
+			(effects
+				(font
+					(size 1.27 1.27)
+				)
+			)
+		)
+		(property "Description" "Resistor, small symbol"
+			(at 231.775 111.76 0)
+			(hide yes)
+			(show_name no)
+			(do_not_autoplace no)
+			(effects
+				(font
+					(size 1.27 1.27)
+				)
+			)
+		)
+		(property "MPN" "C844915"
+			(at 231.775 111.76 90)
+			(hide yes)
+			(show_name no)
+			(do_not_autoplace no)
+			(effects
+				(font
+					(size 1.27 1.27)
+				)
+			)
+		)
+		(pin "2"
+		)
+		(pin "1"
+		)
+		(instances
+			(project "Avionics-MainBoard"
+				(path "/4c932743-8c6f-426e-9c1f-5a3f2b32c70d/1ff82478-f00f-4d48-a429-2ed9117c0498"
+					(reference "R186")
+					(unit 1)
+				)
+			)
+		)
+	)
+	(symbol
 		(lib_id "power:GND")
 		(at 243.84 93.98 0)
@@
 					(unit 1)
 				)
-			)
-		)
-	)
-	(symbol
-		(lib_id "Device:D_Schottky")
-		(at 149.86 111.76 180)
-		(unit 1)
-		(body_style 1)
-		(exclude_from_sim no)
-		(in_bom yes)
-		(on_board yes)
-		(in_pos_files yes)
-		(dnp no)
-		(property "Reference" "D14"
-			(at 149.86 114.935 0)
-			(show_name no)
-			(do_not_autoplace no)
-			(effects
-				(font
-					(size 1.27 1.27)
-				)
-			)
-		)
-		(property "Value" "DFLS130LQ-7"
-			(at 149.86 116.84 0)
-			(show_name no)
-			(do_not_autoplace no)
-			(effects
-				(font
-					(size 1.27 1.27)
-				)
-			)
-		)
-		(property "Footprint" "Diode_SMD:D_PowerDI-123"
-			(at 149.86 111.76 0)
-			(hide yes)
-			(show_name no)
-			(do_not_autoplace no)
-			(effects
-				(font
-					(size 1.27 1.27)
-				)
-			)
-		)
-		(property "Datasheet" ""
-			(at 149.86 111.76 0)
-			(hide yes)
-			(show_name no)
-			(do_not_autoplace no)
-			(effects
-				(font
-					(size 1.27 1.27)
-				)
-			)
-		)
-		(property "Description" "Schottky diode"
-			(at 149.86 111.76 0)
-			(hide yes)
-			(show_name no)
-			(do_not_autoplace no)
-			(effects
-				(font
-					(size 1.27 1.27)
-				)
-			)
-		)
-		(property "MPN" "RB521S30T1G"
-			(at 149.86 104.14 0)
-			(hide yes)
-			(show_name no)
-			(do_not_autoplace no)
-			(effects
-				(font
-					(size 1.27 1.27)
-				)
-				(justify left bottom)
-			)
-		)
-		(property "Manufacturer" "ON Semiconductor"
-			(at 149.86 104.14 0)
-			(hide yes)
-			(show_name no)
-			(do_not_autoplace no)
-			(effects
-				(font
-					(size 1.27 1.27)
-				)
-				(justify left bottom)
-			)
-		)
-		(property "Author" "Antmicro"
-			(at 127 91.44 0)
-			(hide yes)
-			(show_name no)
-			(do_not_autoplace no)
-			(effects
-				(font
-					(size 1.27 1.27)
-					(thickness 0.15)
-				)
-				(justify left bottom)
-			)
-		)
-		(property "License" "Apache-2.0"
-			(at 127 88.9 0)
-			(hide yes)
-			(show_name no)
-			(do_not_autoplace no)
-			(effects
-				(font
-					(size 1.27 1.27)
-					(thickness 0.15)
-				)
-				(justify left bottom)
-			)
-		)
-		(pin "1"
-		)
-		(pin "2"
-		)
-		(instances
-			(project "Avionics-MainBoard"
-				(path "/4c932743-8c6f-426e-9c1f-5a3f2b32c70d/1ff82478-f00f-4d48-a429-2ed9117c0498"
-					(reference "D14")
-					(unit 1)
-				)
