File: I2C_Protection.kicad_sch (KiCad schematic)
At the start: 0 parts

Commit message: Updated version to v2.1
Other:
- company: (none) -> Carnegie Mellon University
- title: (none) -> Argus Mainboard
Changed lines of the file:
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@@
 	(generator_version "8.0")
 	(paper "A4")
+	(title_block
+		(title "Argus Mainboard")
+		(date "2024-11-19")
+		(rev "v2.1")
+		(company "Carnegie Mellon University")
+		(comment 1 "M. Holliday")
+		(comment 2 "N. Khera")
+		(comment 3 "V. Rajesh")
+	)
 	(wire
 		(pts

Commit message: v3 partial schematic updates
Other:
- sheet WireProtection ports: added 3V3; removed none
- sheet WireProtection1 ports: added 3V3; removed none
Changed lines of the file:
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@@
 	(wire
 		(pts
-			(xy 129.54 99.06) (xy 135.89 99.06)
-		)
-		(stroke
-			(width 0)
-			(type default)
-		)
-	)
-	(wire
-		(pts
-			(xy 129.54 85.09) (xy 135.89 85.09)
+			(xy 129.54 85.09) (xy 134.62 85.09)
+		)
+		(stroke
+			(width 0)
+			(type default)
+		)
+	)
+	(wire
+		(pts
+			(xy 129.54 96.52) (xy 134.62 96.52)
+		)
+		(stroke
+			(width 0)
+			(type default)
+		)
+	)
+	(wire
+		(pts
+			(xy 129.54 82.55) (xy 134.62 82.55)
+		)
+		(stroke
+			(width 0)
+			(type default)
+		)
+	)
+	(wire
+		(pts
+			(xy 129.54 99.06) (xy 134.62 99.06)
 		)
 		(stroke
@@
 		)
 	)
+	(hierarchical_label "3V3"
+		(shape bidirectional)
+		(at 129.54 82.55 180)
+		(fields_autoplaced yes)
+		(effects
+			(font
+				(size 1.27 1.27)
+			)
+			(justify right)
+		)
+	)
 	(hierarchical_label "SDA_DEVICE"
 		(shape bidirectional)
@@
 		)
 	)
+	(hierarchical_label "3V3"
+		(shape bidirectional)
+		(at 129.54 96.52 180)
+		(fields_autoplaced yes)
+		(effects
+			(font
+				(size 1.27 1.27)
+			)
+			(justify right)
+		)
+	)
 	(hierarchical_label "SCL_BUS"
 		(shape bidirectional)
@@
 	)
 	(sheet
-		(at 135.89 82.55)
-		(size 16.51 5.08)
+		(at 134.62 80.264)
+		(size 17.78 7.366)
 		(fields_autoplaced yes)
 		(stroke
@@
 		)
 		(property "Sheetname" "WireProtection"
-			(at 135.89 81.8384 0)
+			(at 134.62 79.5524 0)
 			(effects
 				(font
@@
 		)
 		(property "Sheetfile" "WireProtection.kicad_sch"
-			(at 135.89 88.2146 0)
+			(at 134.62 88.2146 0)
 			(effects
 				(font
@@
 		)
 		(pin "DEVICE" bidirectional
-			(at 135.89 85.09 180)
+			(at 134.62 85.09 180)
+			(effects
+				(font
+					(size 1.27 1.27)
+				)
+				(justify left)
+			)
+		)
+		(pin "3V3" input
+			(at 134.62 82.55 180)
 			(effects
 				(font
@@
 					(page "20")
 				)
+				(path "/4c932743-8c6f-426e-9c1f-5a3f2b32c70d/60aa2943-2df4-4541-853f-c25e8e58a8ce/5ab6bffb-ac70-4d04-bc1f-09141586f2fc"
+					(page "19")
+				)
+			)
+			(project ""
+				(path "/6167394f-ef17-4174-a137-33bfda5b3a14/5194385a-96b9-4b1e-ba0c-f9caab4441d8"
+					(page "")
+				)
+			)
+			(project "Avionics-MainBoard"
+				(path "/4c932743-8c6f-426e-9c1f-5a3f2b32c70d/6167394f-ef17-4174-a137-33bfda5b3a14/5194385a-96b9-4b1e-ba0c-f9caab4441d8"
+					(page "6")
+				)
 			)
 		)
 	)
 	(sheet
-		(at 135.89 96.52)
-		(size 16.51 5.08)
+		(at 134.62 93.98)
+		(size 17.78 7.62)
 		(fields_autoplaced yes)
 		(stroke
@@
 		)
 		(property "Sheetname" "WireProtection1"
-			(at 135.89 95.8084 0)
+			(at 134.62 93.2684 0)
 			(effects
 				(font
@@
 		)
 		(property "Sheetfile" "WireProtection.kicad_sch"
-			(at 135.89 102.1846 0)
+			(at 134.62 102.1846 0)
 			(effects
 				(font
@@
 		)
 		(pin "DEVICE" bidirectional
-			(at 135.89 99.06 180)
+			(at 134.62 99.06 180)
+			(effects
+				(font
+					(size 1.27 1.27)
+				)
+				(justify left)
+			)
+		)
+		(pin "3V3" input
+			(at 134.62 96.52 180)
 			(effects
 				(font
@@
 		(instances
 			(project "Avionics-MainBoard"
-				(path "/4c932743-8c6f-426e-9c1f-5a3f2b32c70d/83586450-5275-466d-92ec-f4b550f48d32/1d43a322-a4de-4625-bc76-e4a5abbb5f5f"
-					(page "6")
-				)
 				(path "/4c932743-8c6f-426e-9c1f-5a3f2b32c70d/db13e207-3bf8-4f4b-b8f6-f29c20baff72/fac17611-3490-4577-970c-973f049d9ec4"
 					(page "12")
@@
 					(page "13")
 				)
-				(path "/4c932743-8c6f-426e-9c1f-5a3f2b32c70d/1ff82478-f00f-4d48-a429-2ed9117c0498/6dcdd520-f92f-4264-b446-8551a35308dc"
-					(page "15")
-				)
 				(path "/4c932743-8c6f-426e-9c1f-5a3f2b32c70d/6167394f-ef17-4174-a137-33bfda5b3a14/5194385a-96b9-4b1e-ba0c-f9caab4441d8"
 					(page "16")
@@
 					(page "17")
 				)
-			)
+				(path "/4c932743-8c6f-426e-9c1f-5a3f2b32c70d/60aa2943-2df4-4541-853f-c25e8e58a8ce/5ab6bffb-ac70-4d04-bc1f-09141586f2fc"
+					(page "27")
+				)
+			)
