File: LoRa.kicad_sch (KiCad schematic)
At the start: 20 parts, among them U15 TPS7A4501DCQT, U16 ADM1176-1ARMZ-R7, U7 E22-900M30S

Commit message: v3 partial schematic updates
Parts:
- added C10: 1u, Capacitor_SMD:C_0603_1608Metric, symbol Device:C_Small
- added C13: 22u, Capacitor_SMD:C_1210_3225Metric, symbol Device:C_Small
- added C14: 10n, Capacitor_SMD:C_0603_1608Metric, symbol Device:C_Small
- added R27: 51k, Resistor_SMD:R_0603_1608Metric, symbol Device:R_Small
- added R28: 11k, Resistor_SMD:R_0603_1608Metric, symbol Device:R_Small
- added R29: 1.54k, Resistor_SMD:R_0603_1608Metric, symbol Device:R_Small
- added U2: TPS259621DDA, Package_SO:Texas_R-PDSO-G8_EP2.95x4.9mm_Mask2.4x3.1mm_ThermalVias, symbol oresat-ics:TPS259621DDA
- R112: value ?R -> 0.1R
- R113: value 1K -> 1k
- R43, R44, R45: now not fitted
Connections:
- net GND: now also C10.2, C13.2, C14.2, R28.2, R29.2, U2.1 (GND), U2.9 (GND)
- net VSYS: now also C10.1, C13.1, R27.1, U2.4 (IN); no longer C55.2, U15.2 (IN)
- net VDD_LS: now reaches C56.2, R110.1, R112.2, U15.4 (OUT), U16.1 (VCC)
- net +3V3 renamed +3V3_M
- net LoRa_VDD renamed VDD_LoRa
- new net: C14.1, U2.2 (dVdt)
- new net: R27.2, R28.1, U2.3 (EN/UVLO)
- new net: R29.1, U2.7 (ILM)
- new net VSYS_LoRa: C55.2, U15.2 (IN), U2.5 (OUT)
- no-connect marks 3 -> 5
Other:
- note added: "LoRa Module"
- note added: "LoRa eFuse"
- note added: "Rsense"
- note added: "TODO: INCORRECT ILIM MAYBE CHANGE UVLO USE FLT"
- note added: "TODO: Maybe use ADM1176 GATE + NMOS for OC protection"
- note added: "TPS259621 = Autoretry after thermal shutdown Card current limited to 0.6 A by R_ILM = 1.54k ohm dv/dt = 10nF sets it to 4.2 V/ms instead of the default 70 V/ms OVLO = 13.7 V (open) UVLO = 6.2 V"
- note added: "VSYS 4.5 to 18V"
- note removed: "LoRa #1"
- moved on the sheet: C26, C27, C55, C56, C57, R110, R111, R112, R113, R23, R24, R34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

Commit message: v3 Layout complete
Parts:
- removed R43, R45: 0R, Resistor_SMD:R_0603_1608Metric, symbol Device:R_Small
- added D10, D9: LED_G_0603_LTST-C190GKT, LED_SMD:LED_0603_1608Metric, symbol Device:LED_Small_Filled
- added D11: SZMMSZ5232BT1G, Diode_SMD:D_SOD-123, symbol Device:D_Zener_Small
- added R161, R89: 10k, Resistor_SMD:R_0603_1608Metric, symbol Device:R_Small
- added R90: 4k7, Resistor_SMD:R_0603_1608Metric, symbol Device:R_Small
- C58: renamed from C10; value 1u -> 22u; footprint Capacitor_SMD:C_0603_1608Metric -> Capacitor_SMD:C_1210_3225Metric
- C59: renamed from C13; value 22u -> 1u; footprint Capacitor_SMD:C_1210_3225Metric -> Capacitor_SMD:C_0603_1608Metric
- C61: renamed from C55; footprint Capacitor_SMD:C_0603_1608Metric -> Capacitor_SMD:C_0805_2012Metric
- C62: renamed from C56; footprint Capacitor_SMD:C_0603_1608Metric -> Capacitor_SMD:C_0805_2012Metric
- C87: renamed from C27; value 1u -> 10u; footprint Capacitor_SMD:C_0603_1608Metric -> Capacitor_SMD:C_0805_2012Metric
- R80: renamed from R29; value 1.54k -> 453R
- R82: renamed from R111; value 3.16K -> 3k16
- R83: renamed from R112; value 0.1R -> 0.01R
- R91: renamed from R23; value 10K -> 10k
- R92: renamed from R24; value 10K -> 10k
- R93: renamed from R34; value 10K -> 10k
- R94: renamed from R35; value 10K -> 10k
- U11: renamed from U2; symbol oresat-ics:TPS259621DDA -> Argus-IC:TPS259621DDA
- renumbered C14 to C60, C57 to C63, C26 to C86, R27 to R78, R28 to R79, R110 to R81, R113 to R84, R44 to R86, R53 to R88, U15 to U12, U16 to U13, U7 to U14
Connections:
- net +3V3_M: now also R161.1
- net GND: now also D10.1 (K), D11.2 (A), D9.1 (K)
- net VDD_LS: now also D11.1 (K), R90.2
- net VSYS_LoRa: now also R89.2
- net LoRa_FLT: now reaches U11.6 (*FLT)
- net LoRa_FLT: now also R161.2
- net CSn renamed LoRa_CSn
- new net: D9.2 (A), R89.1
- new net: D10.2 (A), R90.1
- no-connect marks 5 -> 4
Other:
- sheet I2C Protection3 ports: added 3V3; removed none
- note added: "POWER ON"
- note added: "POWER SAFETY"
- note added: "TODO: MAYBE CHANGE UVLO MAYBE CHANGE ILIM"
- note added: "TPS259621 = Autoretry after thermal shutdown Card current limited to 2.0 A by R_ILM = 453 ohm dv/dt = 10nF sets it to 4.2 V/ms instead of the default 70 V/ms OVLO = 13.7 V (open) UVLO = 6.2 V"
- note added: "VGOOD"
- note added: "V_z = 5.6V"
- note removed: "TODO: INCORRECT ILIM MAYBE CHANGE UVLO USE FLT"
- note removed: "TODO: Maybe use ADM1176 GATE + NMOS for OC protection"
- note removed: "TPS259621 = Autoretry after thermal shutdown Card current limited to 0.6 A by R_ILM = 1.54k ohm dv/dt = 10nF sets it to 4.2 V/ms instead of the default 70 V/ms OVLO = 13.7 V (open) UVLO = 6.2 V"
- moved on the sheet: C62

Commit message: Addressed design issues
Other:
- note added: "TODO: MAYBE CHANGE UVLO"
- note removed: "TODO: MAYBE CHANGE UVLO MAYBE CHANGE ILIM"
- moved on the sheet: R86, R88
Changed lines of the file:
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@@
 	(wire
 		(pts
-			(xy 203.2 76.2) (xy 203.2 78.74)
+			(xy 203.2 69.85) (xy 203.2 72.39)
 		)
 		(stroke
@@
 	(wire
 		(pts
-			(xy 218.44 76.2) (xy 218.44 78.74)
+			(xy 218.44 69.85) (xy 218.44 72.39)
 		)
 		(stroke
@@
 	(wire
 		(pts
-			(xy 203.2 83.82) (xy 203.2 86.36)
+			(xy 203.2 77.47) (xy 203.2 80.01)
 		)
 		(stroke
@@
 	(wire
 		(pts
-			(xy 203.2 76.2) (xy 208.28 76.2)
+			(xy 203.2 69.85) (xy 208.28 69.85)
 		)
 		(stroke
@@
 	(wire
 		(pts
-			(xy 218.44 83.82) (xy 218.44 86.36)
+			(xy 218.44 77.47) (xy 218.44 80.01)
 		)
 		(stroke
@@
 	(wire
 		(pts
-			(xy 218.44 76.2) (xy 223.52 76.2)
+			(xy 218.44 69.85) (xy 223.52 69.85)
 		)
 		(stroke
@@
 		)
 	)
-	(text "TODO: MAYBE CHANGE UVLO\nMAYBE CHANGE ILIM\n"
+	(text "TODO: MAYBE CHANGE UVLO"
 		(exclude_from_sim no)
 		(at 38.862 91.44 0)
@@
 	)
 	(label "A0"
-		(at 208.28 76.2 180)
+		(at 208.28 69.85 180)
 		(effects
 			(font
@@
 	)
 	(label "A1"
-		(at 223.52 76.2 180)
+		(at 223.52 69.85 180)
 		(effects
 			(font
@@
 	(symbol
 		(lib_id "power:GND")
-		(at 218.44 86.36 0)
+		(at 218.44 80.01 0)
 		(unit 1)
 		(exclude_from_sim no)
@@
 		(dnp no)
 		(property "Reference" "#PWR0163"
-			(at 218.44 92.71 0)
+			(at 218.44 86.36 0)
 			(effects
 				(font
@@
 		)
 		(property "Value" "GND"
-			(at 218.44 90.17 0)
+			(at 218.44 83.82 0)
 			(effects
 				(font
@@
 		)
 		(property "Footprint" ""
-			(at 218.44 86.36 0)
+			(at 218.44 80.01 0)
 			(effects
 				(font
@@
 		)
 		(property "Datasheet" ""
-			(at 218.44 86.36 0)
+			(at 218.44 80.01 0)
 			(effects
 				(font
@@
 		)
 		(property "Description" "Power symbol creates a global label with name \"GND\" , ground"
-			(at 218.44 86.36 0)
+			(at 218.44 80.01 0)
 			(effects
 				(font
@@
 	(symbol
 		(lib_id "power:GND")
-		(at 203.2 86.36 0)
+		(at 203.2 80.01 0)
 		(unit 1)
 		(exclude_from_sim no)
@@
 		(dnp no)
 		(property "Reference" "#PWR0155"
-			(at 203.2 92.71 0)
+			(at 203.2 86.36 0)
 			(effects
 				(font
@@
 		)
 		(property "Value" "GND"
-			(at 203.2 90.17 0)
+			(at 203.2 83.82 0)
 			(effects
 				(font
@@
 		)
 		(property "Footprint" ""
-			(at 203.2 86.36 0)
+			(at 203.2 80.01 0)
 			(effects
 				(font
@@
 		)
 		(property "Datasheet" ""
-			(at 203.2 86.36 0)
+			(at 203.2 80.01 0)
 			(effects
 				(font
@@
 		)
 		(property "Description" "Power symbol creates a global label with name \"GND\" , ground"
-			(at 203.2 86.36 0)
+			(at 203.2 80.01 0)
 			(effects
 				(font
@@
 	(symbol
 		(lib_id "Device:R_Small")
-		(at 218.44 81.28 0)
+		(at 218.44 74.93 0)
 		(mirror x)
 		(unit 1)
@@
 		(dnp no)
 		(property "Reference" "R88"
-			(at 215.392 80.518 0)
+			(at 215.392 74.168 0)
 			(effects
 				(font
@@
 		)
 		(property "Value" "0R"
-			(at 215.9 82.296 0)
+			(at 215.9 75.946 0)
 			(effects
 				(font
@@
 		)
 		(property "Footprint" "Resistor_SMD:R_0603_1608Metric"
-			(at 218.44 81.28 0)
+			(at 218.44 74.93 0)
 			(effects
 				(font
@@
 		)
 		(property "Datasheet" "~"
-			(at 218.44 81.28 0)
+			(at 218.44 74.93 0)
 			(effects
 				(font
@@
 		)
 		(property "Description" "Resistor, small symbol"
-			(at 218.44 81.28 0)
+			(at 218.44 74.93 0)
 			(effects
 				(font
@@
 	(symbol
 		(lib_id "Device:R_Small")
-		(at 203.2 81.28 0)
+		(at 203.2 74.93 0)
 		(mirror x)
 		(unit 1)
@@
 		(dnp yes)
 		(property "Reference" "R86"
-			(at 200.152 80.518 0)
+			(at 200.152 74.168 0)
 			(effects
 				(font
@@
 		)
 		(property "Value" "0R"
-			(at 200.66 82.296 0)
+			(at 200.66 75.946 0)
 			(effects
 				(font
@@
 		)
 		(property "Footprint" "Resistor_SMD:R_0603_1608Metric"
-			(at 203.2 81.28 0)
+			(at 203.2 74.93 0)
 			(effects
 				(font
@@
 		)
 		(property "Datasheet" "~"
-			(at 203.2 81.28 0)
+			(at 203.2 74.93 0)
 			(effects
 				(font
@@
 		)
 		(property "Description" "Resistor, small symbol"
-			(at 203.2 81.28 0)
+			(at 203.2 74.93 0)
 			(effects
 				(font

Commit message: v4.0 Updates
Parts:
- added R86: 100k, Resistor_SMD:R_0603_1608Metric, symbol Device:R_Small
- renumbered C58 to C56, C59 to C57, C60 to C58, C61 to C59, C62 to C60, C63 to C61, C86 to C64, C87 to C65, D9 to D11, D10 to D12, D11 to D13, R161 to R85, R86 to R87
Connections:
- net GND: now also R86.2
- net LoRa_EN: now also R86.1
Other:
- sheet I2C Protection3 renamed I2C Protection2
- sheet SPI Protection1 renamed SPI Protection
- moved on the sheet: C64, C65, D11, D12, D13, R87, R88, R89, R90, R91, R92, R93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

Commit message: DFM updates
Parts:
- C56: DPN 587-3473-1-ND -> (none); DST Digi-Key -> (none); MFR Taiyo Yuden -> (none); MPN TMK107BJ105KAHT -> C2803395
- C57: DPN 490-GCM32EC71E226KE36KCT-ND -> (none); DST Digi-Key -> (none); MFR Murata Electronics -> (none); MPN GCM32EC71E226KE36K -> C2214844
- C58: DPN 399-14102-1-ND -> (none); DST Digi-Key -> (none); MFR KEMET -> (none); MPN C0603C103J3GECAUTO -> C161232
- C59, C60, C65: MPN (none) -> C386084
- C61: MPN (none) -> C3877267
- C64: MPN (none) -> C2214844
- D11, D12: Author Antmicro -> (none); License Apache-2.0 -> (none); MPN LTST-C190GKT -> C2909774; Manufacturer Lite-On -> (none); Public False -> (none)
- R78: DPN RMCF0603FT10K0CT-ND -> (none); DST Digi-Key -> (none); MFR Stackpole Electronics Inc -> (none); MPN RMCF0603FT10K0 -> C844796
- R79: DPN RMCF0603FT10K0CT-ND -> (none); DST Digi-Key -> (none); MFR Stackpole Electronics Inc -> (none); MPN RMCF0603FT10K0 -> C844734
- R80: DPN RMCF0603FT604RCT-ND -> (none); DST Digi-Key -> (none); MFR Stackpole Electronics Inc -> (none); MPN RMCF0603FT604R -> C278625
- R81: value 10K -> 10k; MPN (none) -> C2479067
- R82: MPN (none) -> C403153
- R83: value 0.01R -> 10m; MPN (none) -> C840621
- R84: MPN (none) -> C2484712
- R85: DPN RMCF0603FT604RCT-ND -> (none); DST Digi-Key -> (none); MFR Stackpole Electronics Inc -> (none); MPN RMCF0603FT604R -> C2479067
- R86: DPN RMCF0603FT604RCT-ND -> (none); DST Digi-Key -> (none); MFR Stackpole Electronics Inc -> (none); MPN RMCF0603FT604R -> C237792
- R87: DNI (none) -> DNI; now left out of the parts list
- R88: MPN (none) -> C844915
- R89: Author Antmicro -> (none); License Apache-2.0 -> (none); MPN CR0402-FX-4701GLF -> C2479067; Manufacturer Bourns -> (none); Tolerance 1% -> (none); Val 4k7 -> (none)
- R90: Author Antmicro -> (none); License Apache-2.0 -> (none); MPN CR0402-FX-4701GLF -> C844931; Manufacturer Bourns -> (none); Tolerance 1% -> (none); Val 4k7 -> (none)
- R91, R92, R93, R94: MPN (none) -> C2479067
- U11: DPN 296-TPS259620DDATCT-ND -> (none); DST Digi-Key -> (none); MFR Texas Instruments -> (none); MPN TPS259620DDAT -> C2155774
- U12: Flight TPS7A4501DCQT -> (none); MPN (none) -> C2869558; Manufacturer_Name Texas Instruments -> (none); Manufacturer_Part_Number TPS7A4501DCQT -> (none); Proto TPS7A4501DCQT -> (none)
- U14: value E22-900M30S -> E22-400M30S; Flight RFM98PW -> (none); MPN (none) -> C411292; Manufacturer_Name HopeRF -> (none); Manufacturer_Part_Number RFM98PW -> (none); Proto RFM98PW -> (none)

Commit message: Minor schematic fixes
Other:
- note added: "Set RF Voltage: VOUT=1.21*(1+R81/R82)+(3E-6*R55) VOUT=5.07V (R81=10K, R82=3.16K)"
- note removed: "Set RF Voltage: VOUT=1.21*(1+R55/R59)+(3E-6*R55) VOUT=5.07V (R55=10K, R59=3.16K)"
Changed lines of the file:
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@@
 		)
 	)
-	(text "Set RF Voltage:\nVOUT=1.21*(1+R55/R59)+(3E-6*R55)\nVOUT=5.07V (R55=10K, R59=3.16K)\n"
+	(text "Set RF Voltage:\nVOUT=1.21*(1+R81/R82)+(3E-6*R55)\nVOUT=5.07V (R81=10K, R82=3.16K)\n"
 		(exclude_from_sim no)
 		(at 116.84 76.962 0)

Commit message: Fixed Jetson FPC pinout
Other:
- note added: "I2C1 ADDR 0x42"
- note removed: "0x42"
- note removed: "I2C1 ADDR"
Changed lines of the file:
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@@
 		)
 	)
-	(text "I2C1 ADDR"
+	(text "I2C1 ADDR\n0x42"
 		(exclude_from_sim no)
-		(at 279.146 76.454 0)
+		(at 261.366 80.01 0)
 		(effects
 			(font
 				(size 2.159 2.159)
 			)
-			(justify right bottom)
+			(justify left bottom)
 		)
 	)
@@
 		)
 	)
-	(text "0x42"
-		(exclude_from_sim no)
-		(at 269.494 80.01 0)
-		(effects
-			(font
-				(size 2.159 2.159)
-			)
-			(justify right bottom)
-		)
-	)

Commit message: v4.2 Updates
Parts:
- added D17: DFLS130LQ-7, Diode_SMD:D_PowerDI-123, symbol Device:D_Schottky_Small
Connections:
- net VSYS_LoRa: now also D17.1 (K)
- new net VUSB: D17.2 (A)
Changed lines of the file:
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@@
 	(title_block
 		(title "Argus Mainboard")
-		(date "2025-01-08")
-		(rev "v3.0")
+		(date "2025-11-24")
+		(rev "v4.2")
 		(company "Carnegie Mellon University")
 		(comment 1 "M. Holliday")
@@
 	(wire
 		(pts
+			(xy 88.9 27.94) (xy 80.01 27.94)
+		)
+		(stroke
+			(width 0)
+			(type default)
+		)
+	)
+	(wire
+		(pts
 			(xy 64.77 54.61) (xy 64.77 63.5)
 		)
@@
 	(wire
 		(pts
+			(xy 93.98 27.94) (xy 102.87 27.94)
+		)
+		(stroke
+			(width 0)
+			(type default)
+		)
+	)
+	(wire
+		(pts
 			(xy 245.11 46.99) (xy 228.6 46.99)
 		)
@@
 	(wire
 		(pts
+			(xy 102.87 25.4) (xy 102.87 27.94)
+		)
+		(stroke
+			(width 0)
+			(type default)
+		)
+	)
+	(wire
+		(pts
 			(xy 104.14 66.04) (xy 100.33 66.04)
 		)
@@
 	(wire
 		(pts
+			(xy 80.01 25.4) (xy 80.01 27.94)
+		)
+		(stroke
+			(width 0)
+			(type default)
+		)
+	)
+	(wire
+		(pts
 			(xy 106.68 138.43) (xy 106.68 139.7)
 		)
@@
 	)
 	(symbol
+		(lib_id "power:+BATT")
+		(at 80.01 25.4 0)
+		(unit 1)
+		(exclude_from_sim no)
+		(in_bom yes)
+		(on_board yes)
+		(dnp no)
+		(property "Reference" "#PWR096"
+			(at 80.01 29.21 0)
+			(effects
+				(font
+					(size 1.27 1.27)
+				)
+				(hide yes)
+			)
+		)
+		(property "Value" "VUSB"
+			(at 80.01 21.59 0)
+			(effects
+				(font
+					(size 1.27 1.27)
+				)
+			)
+		)
+		(property "Footprint" ""
+			(at 80.01 25.4 0)
+			(effects
+				(font
+					(size 1.27 1.27)
+				)
+				(hide yes)
+			)
+		)
+		(property "Datasheet" ""
+			(at 80.01 25.4 0)
+			(effects
+				(font
+					(size 1.27 1.27)
+				)
+				(hide yes)
+			)
+		)
+		(property "Description" "Power symbol creates a global label with name \"+BATT\""
+			(at 80.01 25.4 0)
+			(effects
+				(font
+					(size 1.27 1.27)
+				)
+				(hide yes)
+			)
+		)
+		(pin "1"
+		)
+		(instances
+			(project "Avionics-MainBoard"
+				(path "/4c932743-8c6f-426e-9c1f-5a3f2b32c70d/6167394f-ef17-4174-a137-33bfda5b3a14"
+					(reference "#PWR096")
+					(unit 1)
+				)
+			)
+		)
+	)
+	(symbol
 		(lib_id "power:GND")
 		(at 200.66 93.98 0)
@@
 	)
 	(symbol
+		(lib_id "power:+BATT")
+		(at 102.87 25.4 0)
+		(unit 1)
+		(exclude_from_sim no)
+		(in_bom yes)
+		(on_board yes)
+		(dnp no)
+		(property "Reference" "#PWR0107"
+			(at 102.87 29.21 0)
+			(effects
+				(font
+					(size 1.27 1.27)
+				)
+				(hide yes)
+			)
+		)
+		(property "Value" "VSYS_LoRa"
+			(at 102.87 21.59 0)
+			(effects
+				(font
+					(size 1.27 1.27)
+				)
+			)
+		)
+		(property "Footprint" ""
+			(at 102.87 25.4 0)
+			(effects
+				(font
+					(size 1.27 1.27)
+				)
+				(hide yes)
+			)
+		)
+		(property "Datasheet" ""
+			(at 102.87 25.4 0)
+			(effects
+				(font
+					(size 1.27 1.27)
+				)
+				(hide yes)
+			)
+		)
+		(property "Description" "Power symbol creates a global label with name \"+BATT\""
+			(at 102.87 25.4 0)
+			(effects
+				(font
+					(size 1.27 1.27)
+				)
+				(hide yes)
+			)
+		)
+		(pin "1"
+		)
+		(instances
+			(project "Avionics-MainBoard"
+				(path "/4c932743-8c6f-426e-9c1f-5a3f2b32c70d/6167394f-ef17-4174-a137-33bfda5b3a14"
+					(reference "#PWR0107")
+					(unit 1)
+				)
+			)
+		)
+	)
+	(symbol
 		(lib_id "power:GND")
 		(at 177.8 93.98 0)
@@
 					(unit 1)
 				)
+			)
+		)
+	)
+	(symbol
+		(lib_id "Device:D_Schottky_Small")
+		(at 91.44 27.94 180)
+		(unit 1)
+		(exclude_from_sim no)
+		(in_bom yes)
+		(on_board yes)
+		(dnp no)
+		(property "Reference" "D17"
+			(at 91.44 23.368 0)
+			(effects
+				(font
+					(size 1.27 1.27)
+				)
+			)
+		)
+		(property "Value" "DFLS130LQ-7"
+			(at 91.44 25.4 0)
+			(effects
+				(font
+					(size 1.27 1.27)
+				)
+			)
+		)
+		(property "Footprint" "Diode_SMD:D_PowerDI-123"
+			(at 91.44 27.94 90)
+			(effects
+				(font
+					(size 1.27 1.27)
+				)
+				(hide yes)
+			)
+		)
+		(property "Datasheet" "~"
+			(at 91.44 27.94 90)
+			(effects
+				(font
+					(size 1.27 1.27)
+				)
+				(hide yes)
+			)
+		)
+		(property "Description" ""
+			(at 91.44 27.94 0)
+			(effects
+				(font
+					(size 1.27 1.27)
+				)
+			)
+		)
+		(pin "1"
+		)
+		(pin "2"
+		)
+		(instances
+			(project "Avionics-MainBoard"
+				(path "/4c932743-8c6f-426e-9c1f-5a3f2b32c70d/6167394f-ef17-4174-a137-33bfda5b3a14"
+					(reference "D17")
+					(unit 1)
+				)
