File: LoRa.kicad_sch (KiCad schematic)
At the start: 33 parts, among them U11 TPS259621DDA, U12 TPS7A4501DCQT, U13 ADM1176-1ARMZ-R7, U14 E22-400M30S

Commit message: v5.0 Updates
Parts:
- removed C61: 3n3, Capacitor_SMD:C_0603_1608Metric, symbol Device:C_Small
- removed D11: LED_G_0603_LTST-C190GKT, LED_SMD:LED_0603_1608Metric, symbol Device:LED_Small_Filled
- removed D17: DFLS130LQ-7, Diode_SMD:D_PowerDI-123, symbol Device:D_Schottky_Small
- removed R83: 10m, Resistor_SMD:R_2512_6332Metric, symbol Device:R_Small
- removed U11: TPS259621DDA, Package_SO:Texas_R-PDSO-G8_EP2.95x4.9mm_Mask2.4x3.1mm_ThermalVias, symbol Argus-IC:TPS259621DDA
- removed U12: TPS7A4501DCQT, Package_TO_SOT_SMD:SOT-223-6, symbol Argus-IC:TPS7A4501DCQT
- removed U13: ADM1176-1ARMZ-R7, Package_SO:MSOP-10_3x3mm_P0.5mm, symbol Argus-IC:ADM1176-1ARMZ-R7
- added C51, C52: 10u, Capacitor_SMD:C_0805_2012Metric, symbol Device:C_Small
- added C53: 3n3, Capacitor_SMD:C_0603_1608Metric, symbol Device:C_Small
- added C54, C55: 22u, Capacitor_SMD:C_1210_3225Metric, symbol Device:C_Small
- added J11: 60612202111308, Argus-Connectors:60612202111308, symbol Connector:Conn_Coaxial_Small
- added L4: 2.2uH, Inductor_SMD:L_Coilcraft_XAL4020-XXX, symbol Device:L
- added R25, R90, R91, R92: 0R, Resistor_SMD:R_0603_1608Metric, symbol Device:R_Small
- added R86: 10m, Resistor_SMD:R_1206_3216Metric, symbol Device:R_Small
- added TP6, TP7: TestPoint, TestPoint:TestPoint_Pad_D1.5mm, symbol Connector:TestPoint
- added U10: TPS62902QRYTRQ1, Argus-IC:TPS62902QRYTRQ1, symbol Argus-IC:TPS62902QRYTRQ1
- added U11: TPS7A52-Q1, Argus-IC:TPS7A5201Q, symbol Argus-IC:TPS7A52-Q1
- added U12: INA226-Q1, Package_SO:TSSOP-10_3x3mm_P0.5mm, symbol Sensor_Energy:INA226
- C56: value 22u -> 10u; footprint Capacitor_SMD:C_1210_3225Metric -> Capacitor_SMD:C_0805_2012Metric
- C57: value 1u -> 10n; MPN C2214844 -> C2803395
- C58: MPN C161232 -> C2803395
- C59: value 10u -> 22u; footprint Capacitor_SMD:C_0805_2012Metric -> Capacitor_SMD:C_1210_3225Metric; MPN C386084 -> C2803395
- C60: value 10u -> 100n; footprint Capacitor_SMD:C_0805_2012Metric -> Capacitor_SMD:C_0603_1608Metric; MPN C386084 -> C2803395
- C63: renamed from C64; value 1u -> 100u; footprint Capacitor_SMD:C_0603_1608Metric -> Capacitor_SMD:C_1210_3225Metric
- C64: renamed from C65; value 10u -> 100u; footprint Capacitor_SMD:C_0805_2012Metric -> Capacitor_SMD:C_1210_3225Metric
- D12: renamed from D13; now not fitted; now left out of the parts list
- R78: value 51k -> 11k; MPN C844796 -> C844759
- R79: value 11k -> 0R; MPN C844734 -> C844759
- R80: value 453R -> 10k; MPN C278625 -> C844759
- R81: value 10k -> 120k; MPN C2479067 -> C844759
- R82: value 3k16 -> 15k; MPN C403153 -> C844759
- R84: value 1k -> 12k1; MPN C2484712 -> C844759
- R85: value 10k -> 2k23; MPN C2479067 -> C844759
- R87: DNI DNI -> (none); MPN (none) -> C237792
- R88: MPN C844915 -> C237792
- R89: value 10k -> 0R; MPN C2479067 -> C844915; now not fitted; now left out of the parts list
- U13: renamed from U14; value E22-400M30S -> E22P-433M30S; MPN C411292 -> (none)
- renumbered D12 to D11, R90 to R105, R91 to R106, R92 to R107, R93 to R108, R94 to R109, R86 to R83
Connections:
- net LoRa_FLT is gone; now on an unnamed net: R85.2
- net +3V3_M: now also R87.1; no longer R85.1
- net +3V3_P: now also R88.1
- net A0: now also R89.1, R91.2, U12.2 (A0); no longer R87.2
- net A1: now also R90.1, R92.2, U12.1 (A1); no longer R88.2
- net GND: now also C56.1, C57.1, R78.1, R82.1, R85.1, C51.2, C52.2, C53.1, C54.1, C55.1, J11.2 (Ext), R91.1, R92.1, U10.4 (GND), U11.18 (GND), U11.21 (PAD_GND), U11.8 (GND), U12.7 (GND); no longer C56.2, C57.2, C58.2, R79.2, R80.2, R82.2, R87.1, R88.1
- net I2C Protection2/SCL_DEVICE: now also U12.5 (SCL)
- net I2C Protection2/SDA_DEVICE: now also U12.4 (SDA)
- net LoRa_EN: now also U10.5 (EN)
- net VDD_LoRa: now also R86.1, U12.8 (Vbus), U12.9 (Vin-); no longer R84.1
- net VSYS: now also C51.1, C52.1, U10.6 (VIN); no longer C56.1, C57.1, R78.1
- net VSYS_LoRa: now also C58.2, D12.1 (K), R105.2, R84.2, R25.1, R86.2, TP7.1, U11.1 (OUT), U11.19 (OUT), U11.20 (OUT), U12.10 (Vin+); no longer R89.2
- net IN: now reaches R81.2
- net IN: now also C56.2, R80.2, C54.2, C55.2, L4.2, R25.2, TP6.1, U10.3 (VOS), U11.15 (IN), U11.16 (IN), U11.17 (IN); no longer R82.1
- net at C58.1: now also R84.1, U11.3 (FB)
- net at R78.2: now also U10.7 (MODE/S-CONF); no longer R79.1
- net Preg_PG: now reaches R80.1
- net Preg_PG: now also R79.1, U11.14 (EN)
- net at U13.21 (ANT): now also J11.1 (In)
- removed net VDD_LS: C60.2, D12.1 (K), R105.2, R81.1
- new net: C57.2, U11.13 (NR/SS)
- new net: R79.2, U10.1 (PG)
- new net: R81.1, R82.2, U10.9 (FB/VSET)
- new net: C53.2, U10.8 (SS/TR)
- new net: U11.10 (NC), U11.11 (NC), U11.2 (NC), U11.5 (DNC), U11.6 (NC), U11.7 (NC), U11.9 (NC)
- new net: L4.1, U10.2 (SW)
- new net VDD_L: C60.2, R87.2, R88.2, R89.2, R90.2, U12.6 (VS)
Other:
- note added: "I2C1 ADDR 0x44"
- note added: "LoRa LDO"
- note added: "LoRa Pre-Regulator"
- note added: "R81 = R82 * (VOUT / 0.6 - 1) VOUT = 5.4V"
- note added: "Set RF Voltage: VOUT=0.8*(1+R84/R85) VOUT=5.14V (R84=12.1K, R85=2.23K)"
- note added: "SmartConfig R_{mode} = 11k FB/VSET Pin: External FB F{SW}(MHz): 1MHz Output discharge: yes Mode: Auto PFM / PWM"
- note added: "Soft Start C_{ss} = T_{ss} * I_{ss} / V{ref} I_{ss} = 2.5uA V_{ref} = V_{FB} / 0.75 = 0.6 / 0.75"
- note removed: "I2C1 ADDR 0x42"
- note removed: "LoRa Regulator"
- note removed: "LoRa eFuse"
- note removed: "Set RF Voltage: VOUT=1.21*(1+R81/R82)+(3E-6*R55) VOUT=5.07V (R81=10K, R82=3.16K)"
- note removed: "TODO: MAYBE CHANGE UVLO"
- note removed: "TPS259621 = Autoretry after thermal shutdown Card current limited to 2.0 A by R_ILM = 453 ohm dv/dt = 10nF sets it to 4.2 V/ms instead of the default 70 V/ms OVLO = 13.7 V (open) UVLO = 6.2 V"
- note removed: "VGOOD"
- note removed: "VSYS 4.5 to 18V"
- moved on the sheet: C63, C64, D11, R105, R106, R107, R108, R109, R83, U13

Commit message: Final v5.0 Release
Parts:
- R106, R107: value 10k -> 100k
Connections:
- net PG_LoRa: now reaches U11.4 (PG)
- net PG_LoRa: now also D11.2 (A), R105.1
- no-connect marks 4 -> 3
Other:
- moved on the sheet: R86
Changed lines of the file:
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@@
 	(text "Rsense"
 		(exclude_from_sim no)
-		(at 63.627 109.474 90)
+		(at 61.595 109.22 90)
 		(effects
 			(font
@@
 	)
 	(junction
-		(at 61.595 104.14)
+		(at 59.69 104.14)
 		(diameter 0)
 		(color 0 0 0 0)
@@
 	)
 	(junction
-		(at 61.595 114.3)
+		(at 59.69 114.3)
 		(diameter 0)
 		(color 0 0 0 0)
@@
 	)
 	(junction
+		(at 221.615 104.14)
+		(diameter 0)
+		(color 0 0 0 0)
+	)
+	(junction
 		(at 66.675 163.195)
 		(diameter 0)
@@
 		(at 92.71 113.03)
 	)
-	(no_connect
-		(at 237.49 37.465)
-	)
 	(wire
 		(pts
@@
 	(wire
 		(pts
-			(xy 52.705 120.65) (xy 52.705 118.11)
+			(xy 50.8 120.65) (xy 50.8 118.11)
 		)
 		(stroke
@@
 	(wire
 		(pts
-			(xy 67.945 110.49) (xy 67.945 114.3)
+			(xy 71.12 110.49) (xy 71.12 114.3)
 		)
 		(stroke
@@
 	(wire
 		(pts
+			(xy 59.69 104.14) (xy 71.12 104.14)
+		)
+		(stroke
+			(width 0)
+			(type default)
+		)
+	)
+	(wire
+		(pts
 			(xy 177.165 128.27) (xy 177.165 130.81)
 		)
@@
 	(wire
 		(pts
-			(xy 72.39 91.44) (xy 72.39 97.79)
+			(xy 71.12 91.44) (xy 71.12 97.79)
 		)
 		(stroke
@@
 	(wire
 		(pts
-			(xy 61.595 111.76) (xy 61.595 114.3)
+			(xy 59.69 111.76) (xy 59.69 114.3)
 		)
 		(stroke
@@
 	(wire
 		(pts
-			(xy 67.945 107.95) (xy 67.945 104.14)
+			(xy 71.12 107.95) (xy 71.12 104.14)
 		)
 		(stroke
@@
 	(wire
 		(pts
-			(xy 221.615 102.235) (xy 221.615 106.045)
+			(xy 221.615 102.235) (xy 221.615 104.14)
 		)
 		(stroke
@@
 	(wire
 		(pts
-			(xy 61.595 104.14) (xy 61.595 106.68)
+			(xy 59.69 104.14) (xy 59.69 106.68)
 		)
 		(stroke
@@
 	(wire
 		(pts
+			(xy 59.69 114.3) (xy 71.12 114.3)
+		)
+		(stroke
+			(width 0)
+			(type default)
+		)
+	)
+	(wire
+		(pts
 			(xy 156.845 190.5) (xy 169.545 190.5)
 		)
@@
 	(wire
 		(pts
-			(xy 67.945 104.14) (xy 61.595 104.14)
+			(xy 237.49 37.465) (xy 247.015 37.465)
 		)
 		(stroke
@@
 	(wire
 		(pts
-			(xy 61.595 120.65) (xy 61.595 114.3)
+			(xy 59.69 120.65) (xy 59.69 114.3)
 		)
 		(stroke
@@
 	(wire
 		(pts
+			(xy 213.36 104.14) (xy 221.615 104.14)
+		)
+		(stroke
+			(width 0)
+			(type default)
+		)
+	)
+	(wire
+		(pts
 			(xy 113.03 33.655) (xy 113.03 28.575)
 		)
@@
 	(wire
 		(pts
+			(xy 221.615 104.14) (xy 221.615 106.045)
+		)
+		(stroke
+			(width 0)
+			(type default)
+		)
+	)
+	(wire
+		(pts
 			(xy 90.805 178.435) (xy 90.805 180.975)
 		)
@@
 	(wire
 		(pts
+			(xy 71.12 97.79) (xy 72.39 97.79)
+		)
+		(stroke
+			(width 0)
+			(type default)
+		)
+	)
+	(wire
+		(pts
 			(xy 88.265 188.595) (xy 88.265 178.435)
 		)
@@
 	(wire
 		(pts
-			(xy 52.705 120.65) (xy 61.595 120.65)
+			(xy 50.8 120.65) (xy 59.69 120.65)
 		)
 		(stroke
@@
 	(wire
 		(pts
-			(xy 72.39 110.49) (xy 67.945 110.49)
+			(xy 72.39 110.49) (xy 71.12 110.49)
 		)
 		(stroke
@@
 	(wire
 		(pts
-			(xy 67.945 114.3) (xy 61.595 114.3)
-		)
-		(stroke
-			(width 0)
-			(type default)
-		)
-	)
-	(wire
-		(pts
 			(xy 85.725 178.435) (xy 85.725 180.975)
 		)
@@
 	(wire
 		(pts
-			(xy 61.595 91.44) (xy 61.595 104.14)
+			(xy 59.69 91.44) (xy 59.69 104.14)
 		)
 		(stroke
@@
 	(wire
 		(pts
-			(xy 72.39 107.95) (xy 67.945 107.95)
+			(xy 72.39 107.95) (xy 71.12 107.95)
 		)
 		(stroke
@@
 		)
 	)
+	(label "PG_LoRa"
+		(at 247.015 37.465 180)
+		(effects
+			(font
+				(size 1.27 1.27)
+			)
+			(justify right bottom)
+		)
+	)
 	(label "LoRa_CSn"
 		(at 255.27 146.685 0)
@@
 		)
 	)
+	(label "PG_LoRa"
+		(at 213.36 104.14 0)
+		(effects
+			(font
+				(size 1.27 1.27)
+			)
+			(justify left bottom)
+		)
+	)
 	(label "LoRa_RX_EN"
 		(at 41.275 168.275 0)
@@
 	(symbol
 		(lib_id "power:+BATT")
-		(at 72.39 91.44 0)
+		(at 71.12 91.44 0)
 		(unit 1)
 		(body_style 1)
@@
 		(dnp no)
 		(property "Reference" "#PWR0155"
-			(at 72.39 95.25 0)
+			(at 71.12 95.25 0)
 			(hide yes)
 			(show_name no)
@@
 		)
 		(property "Value" "VDD_LoRa"
-			(at 72.39 87.63 0)
+			(at 71.12 87.63 0)
 			(show_name no)
 			(do_not_autoplace no)
@@
 		)
 		(property "Footprint" ""
-			(at 72.39 91.44 0)
+			(at 71.12 91.44 0)
 			(hide yes)
 			(show_name no)
@@
 		)
 		(property "Datasheet" ""
-			(at 72.39 91.44 0)
+			(at 71.12 91.44 0)
 			(hide yes)
 			(show_name no)
@@
 		)
 		(property "Description" "Power symbol creates a global label with name \"+BATT\""
-			(at 72.39 91.44 0)
+			(at 71.12 91.44 0)
 			(hide yes)
 			(show_name no)
@@
 	(symbol
 		(lib_id "power:+BATT")
-		(at 52.705 118.11 0)
+		(at 50.8 118.11 0)
 		(unit 1)
 		(body_style 1)
@@
 		(dnp no)
 		(property "Reference" "#PWR0144"
-			(at 52.705 121.92 0)
+			(at 50.8 121.92 0)
 			(hide yes)
 			(show_name no)
@@
 		)
 		(property "Value" "VDD_LoRa"
-			(at 52.705 114.3 0)
+			(at 50.8 114.3 0)
 			(show_name no)
 			(do_not_autoplace no)
@@
 		)
 		(property "Footprint" ""
-			(at 52.705 118.11 0)
+			(at 50.8 118.11 0)
 			(hide yes)
 			(show_name no)
@@
 		)
 		(property "Datasheet" ""
-			(at 52.705 118.11 0)
+			(at 50.8 118.11 0)
 			(hide yes)
 			(show_name no)
@@
 		)
 		(property "Description" "Power symbol creates a global label with name \"+BATT\""
-			(at 52.705 118.11 0)
+			(at 50.8 118.11 0)
 			(hide yes)
 			(show_name no)
@@
 	(symbol
 		(lib_id "Device:R_Small")
-		(at 61.595 109.22 0)
+		(at 59.69 109.22 0)
 		(mirror x)
 		(unit 1)
@@
 		(dnp no)
 		(property "Reference" "R86"
-			(at 60.325 108.204 0)
+			(at 58.42 108.204 0)
 			(show_name no)
 			(do_not_autoplace no)
@@
 		)
 		(property "Value" "10m"
-			(at 60.325 110.49 0)
+			(at 58.42 110.49 0)
 			(show_name no)
 			(do_not_autoplace no)
@@
 		)
 		(property "Footprint" "Resistor_SMD:R_1206_3216Metric"
-			(at 61.595 109.22 0)
+			(at 59.69 109.22 0)
 			(hide yes)
 			(show_name no)
@@
 		)
 		(property "Datasheet" ""
-			(at 61.595 109.22 0)
+			(at 59.69 109.22 0)
 			(hide yes)
 			(show_name no)
@@
 		)
 		(property "Description" "Resistor, small symbol"
-			(at 61.595 109.22 0)
+			(at 59.69 109.22 0)
 			(hide yes)
 			(show_name no)
@@
 		)
 		(property "MPN" "C840621"
-			(at 61.595 109.22 0)
+			(at 59.69 109.22 0)
 			(hide yes)
 			(show_name no)
@@
 	(symbol
 		(lib_id "power:+BATT")
-		(at 61.595 91.44 0)
+		(at 59.69 91.44 0)
 		(unit 1)
 		(body_style 1)
@@
 		(dnp no)
 		(property "Reference" "#PWR044"
-			(at 61.595 95.25 0)
+			(at 59.69 95.25 0)
 			(hide yes)
 			(show_name no)
@@
 		)
 		(property "Value" "VSYS_LoRa"
-			(at 61.595 87.63 0)
+			(at 59.69 87.63 0)
 			(show_name no)
 			(do_not_autoplace no)
@@
 		)
 		(property "Footprint" ""
-			(at 61.595 91.44 0)
+			(at 59.69 91.44 0)
 			(hide yes)
 			(show_name no)
@@
 		)
 		(property "Datasheet" ""
-			(at 61.595 91.44 0)
+			(at 59.69 91.44 0)
 			(hide yes)
 			(show_name no)
@@
 		)
 		(property "Description" "Power symbol creates a global label with name \"+BATT\""
-			(at 61.595 91.44 0)
+			(at 59.69 91.44 0)
 			(hide yes)
 			(show_name no)
@@
 			)
 		)
-		(property "Value" "10k"
+		(property "Value" "100k"
 			(at 53.34 178.181 0)
 			(show_name no)
@@
 			)
 		)
-		(property "Value" "10k"
+		(property "Value" "100k"
 			(at 60.325 178.181 0)
 			(show_name no)
