File: SPI_Protection.kicad_sch (KiCad schematic)
At the start: 5 parts, among them Q14 MMBT2907

Commit message: v1 done
Parts:
- Q14: symbol Mainboard:MMBT2907 -> Transistor_BJT:MMBTA56
Changed lines of the file:
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@@
 	)
 	(symbol
-		(lib_id "Mainboard:MMBT2907")
+		(lib_id "Transistor_BJT:MMBTA56")
 		(at 120.65 97.79 270)
 		(unit 1)
@@
 		)
 		(property "Footprint" "Package_TO_SOT_SMD:SOT-23"
-			(at 106.426 101.6 0)
+			(at 118.745 102.87 0)
+			(effects
+				(font
+					(size 1.27 1.27)
+					(italic yes)
+				)
+				(justify left)
+				(hide yes)
+			)
+		)
+		(property "Datasheet" "https://diotec.com/request/datasheet/mmbta56.pdf"
+			(at 120.65 97.79 0)
 			(effects
 				(font
 					(size 1.27 1.27)
 				)
+				(justify left)
 				(hide yes)
 			)
 		)
-		(property "Datasheet" ""
-			(at 101.6 111.506 0)
+		(property "Description" "0.5A Ic, 80V Vce, general purpose PNP"
+			(at 120.65 99.06 0)
 			(effects
 				(font
-					(size 1.27 1.27)
-				)
-				(hide yes)
-			)
-		)
-		(property "Description" "PNP BJT - PNP"
-			(at 120.65 97.79 0)
-			(effects
-				(font

Commit message: Updated version to v2.1
Other:
- company: (none) -> Carnegie Mellon University
- title: (none) -> Argus Mainboard
Changed lines of the file:
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@@
 	(generator_version "8.0")
 	(paper "A4")
+	(title_block
+		(title "Argus Mainboard")
+		(date "2024-11-19")
+		(rev "v2.1")
+		(company "Carnegie Mellon University")
+		(comment 1 "M. Holliday")
+		(comment 2 "N. Khera")
+		(comment 3 "V. Rajesh")
+	)
 	(wire
 		(pts

Commit message: v3 partial schematic updates
Parts:
- R50: value 4.7K -> 4.7k
- R51, R52: value 1K -> 1k
Other:
- moved on the sheet: R49, R50
Changed lines of the file:
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@@
 	(wire
 		(pts
-			(xy 176.53 91.44) (xy 177.8 91.44)
-		)
-		(stroke
-			(width 0)
-			(type default)
-		)
-	)
-	(wire
-		(pts
-			(xy 176.53 100.33) (xy 177.8 100.33)
-		)
-		(stroke
-			(width 0)
-			(type default)
-		)
-	)
-	(wire
-		(pts
-			(xy 114.3 100.33) (xy 115.57 100.33)
-		)
-		(stroke
-			(width 0)
-			(type default)
-		)
-	)
-	(wire
-		(pts
-			(xy 127 100.33) (xy 125.73 100.33)
-		)
-		(stroke
-			(width 0)
-			(type default)
-		)
-	)
-	(wire
-		(pts
-			(xy 107.95 100.33) (xy 109.22 100.33)
-		)
-		(stroke
-			(width 0)
-			(type default)
-		)
-	)
-	(wire
-		(pts
-			(xy 170.18 91.44) (xy 171.45 91.44)
-		)
-		(stroke
-			(width 0)
-			(type default)
-		)
-	)
-	(wire
-		(pts
-			(xy 113.03 92.71) (xy 114.3 92.71)
-		)
-		(stroke
-			(width 0)
-			(type default)
-		)
-	)
-	(wire
-		(pts
-			(xy 119.38 92.71) (xy 120.65 92.71)
-		)
-		(stroke
-			(width 0)
-			(type default)
-		)
-	)
-	(wire
-		(pts
-			(xy 170.18 100.33) (xy 171.45 100.33)
+			(xy 176.53 91.44) (xy 179.07 91.44)
+		)
+		(stroke
+			(width 0)
+			(type default)
+		)
+	)
+	(wire
+		(pts
+			(xy 176.53 100.33) (xy 179.07 100.33)
+		)
+		(stroke
+			(width 0)
+			(type default)
+		)
+	)
+	(wire
+		(pts
+			(xy 113.03 100.33) (xy 115.57 100.33)
+		)
+		(stroke
+			(width 0)
+			(type default)
+		)
+	)
+	(wire
+		(pts
+			(xy 128.27 100.33) (xy 125.73 100.33)
+		)
+		(stroke
+			(width 0)
+			(type default)
+		)
+	)
+	(wire
+		(pts
+			(xy 105.41 100.33) (xy 107.95 100.33)
+		)
+		(stroke
+			(width 0)
+			(type default)
+		)
+	)
+	(wire
+		(pts
+			(xy 168.91 91.44) (xy 171.45 91.44)
+		)
+		(stroke
+			(width 0)
+			(type default)
+		)
+	)
+	(wire
+		(pts
+			(xy 120.65 91.44) (xy 120.65 92.71)
+		)
+		(stroke
+			(width 0)
+			(type default)
+		)
+	)
+	(wire
+		(pts
+			(xy 105.41 91.44) (xy 110.49 91.44)
+		)
+		(stroke
+			(width 0)
+			(type default)
+		)
+	)
+	(wire
+		(pts
+			(xy 115.57 91.44) (xy 120.65 91.44)
+		)
+		(stroke
+			(width 0)
+			(type default)
+		)
+	)
+	(wire
+		(pts
+			(xy 168.91 100.33) (xy 171.45 100.33)
 		)
 		(stroke
@@
 	(hierarchical_label "MOSI_Master"
 		(shape input)
-		(at 170.18 100.33 180)
+		(at 168.91 100.33 180)
 		(fields_autoplaced yes)
 		(effects
@@
 	(hierarchical_label "MOSI_Slave"
 		(shape output)
-		(at 177.8 100.33 0)
+		(at 179.07 100.33 0)
 		(fields_autoplaced yes)
 		(effects
@@
 	(hierarchical_label "CLK_Slave"
 		(shape output)
-		(at 177.8 91.44 0)
+		(at 179.07 91.44 0)
 		(fields_autoplaced yes)
 		(effects
@@
 	(hierarchical_label "MISO_Slave"
 		(shape input)
-		(at 107.95 100.33 180)
+		(at 105.41 100.33 180)
 		(fields_autoplaced yes)
 		(effects
@@
 	(hierarchical_label "CSn"
 		(shape input)
-		(at 113.03 92.71 180)
+		(at 105.41 91.44 180)
 		(fields_autoplaced yes)
 		(effects
@@
 	(hierarchical_label "MISO_Master"
 		(shape output)
-		(at 127 100.33 0)
+		(at 128.27 100.33 0)
 		(fields_autoplaced yes)
 		(effects
@@
 	(hierarchical_label "CLK_Master"
 		(shape input)
-		(at 170.18 91.44 180)
+		(at 168.91 91.44 180)
 		(fields_autoplaced yes)
 		(effects
@@
 	(symbol
 		(lib_id "Device:R_Small")
-		(at 116.84 92.71 270)
+		(at 113.03 91.44 270)
 		(unit 1)
 		(exclude_from_sim no)
@@
 		(dnp no)
 		(property "Reference" "R50"
-			(at 116.84 88.646 90)
-			(effects
-				(font
-					(size 1.27 1.27)
-				)
-			)
-		)
-		(property "Value" "4.7K"
-			(at 116.84 90.678 90)
+			(at 113.03 87.376 90)
+			(effects
+				(font
+					(size 1.27 1.27)
+				)
+			)
+		)
+		(property "Value" "4.7k"
+			(at 113.03 89.408 90)
 			(effects
 				(font
@@
 		)
 		(property "Footprint" "Resistor_SMD:R_0603_1608Metric"
-			(at 116.84 92.71 0)
+			(at 113.03 91.44 0)
 			(effects
 				(font
@@
 		)
 		(property "Datasheet" "~"
-			(at 116.84 92.71 0)
+			(at 113.03 91.44 0)
 			(effects
 				(font
@@
 		)
 		(property "Description" "Resistor, small symbol"
-			(at 116.84 92.71 0)
+			(at 113.03 91.44 0)
 			(effects
 				(font
@@
 			)
 		)
-		(property "Value" "1K"
+		(property "Value" "1k"
 			(at 173.99 98.044 90)
 			(effects
@@
 			)
 		)
-		(property "Value" "1K"
+		(property "Value" "1k"
 			(at 173.99 89.154 90)
 			(effects
@@
 	(symbol
 		(lib_id "Device:R_Small")
-		(at 111.76 100.33 270)
+		(at 110.49 100.33 270)
 		(unit 1)
 		(exclude_from_sim no)
@@
 		(dnp no)
 		(property "Reference" "R49"
-			(at 111.76 96.52 90)
+			(at 110.49 96.52 90)
 			(effects
 				(font
@@
 		)
 		(property "Value" "0R"
-			(at 111.76 98.298 90)
+			(at 110.49 98.298 90)
 			(effects
 				(font
@@
 		)
 		(property "Footprint" "Resistor_SMD:R_0603_1608Metric"
-			(at 111.76 100.33 0)
+			(at 110.49 100.33 0)
 			(effects
 				(font
@@
 		)
 		(property "Datasheet" "~"
-			(at 111.76 100.33 0)
+			(at 110.49 100.33 0)
 			(effects
 				(font
@@
 		)
 		(property "Description" "Resistor, small symbol"
-			(at 111.76 100.33 0)
-			(effects
-				(font
+			(at 110.49 100.33 0)
+			(effects
+				(font

Commit message: v3 Layout complete
Parts:
- added R133: 0R, Resistor_SMD:R_0603_1608Metric, symbol Device:R_Small
- R129: renamed from R50; value 4.7k -> 4k7
- renumbered Q14 to Q18, R49 to R130, R51 to R131, R52 to R132
Connections:
- net MISO_Master: now also R133.1
- net MISO_Slave: now also R133.2
Changed lines of the file:
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@@
 	(title_block
 		(title "Argus Mainboard")
-		(date "2024-11-19")
-		(rev "v2.1")
+		(date "2025-01-08")
+		(rev "v3.0")
 		(company "Carnegie Mellon University")
 		(comment 1 "M. Holliday")
@@
 	(wire
 		(pts
+			(xy 168.91 109.22) (xy 171.45 109.22)
+		)
+		(stroke
+			(width 0)
+			(type default)
+		)
+	)
+	(wire
+		(pts
 			(xy 115.57 91.44) (xy 120.65 91.44)
+		)
+		(stroke
+			(width 0)
+			(type default)
+		)
+	)
+	(wire
+		(pts
+			(xy 176.53 109.22) (xy 179.07 109.22)
 		)
 		(stroke
@@
 		(shape input)
 		(at 168.91 100.33 180)
-		(fields_autoplaced yes)
 		(effects
 			(font
@@
 		(shape output)
 		(at 179.07 100.33 0)
-		(fields_autoplaced yes)
 		(effects
 			(font
@@
 		(shape output)
 		(at 179.07 91.44 0)
-		(fields_autoplaced yes)
 		(effects
 			(font
@@
 		(shape input)
 		(at 105.41 100.33 180)
-		(fields_autoplaced yes)
 		(effects
 			(font
@@
 		(shape input)
 		(at 105.41 91.44 180)
-		(fields_autoplaced yes)
 		(effects
 			(font
@@
 		(shape output)
 		(at 128.27 100.33 0)
-		(fields_autoplaced yes)
 		(effects
 			(font
@@
 			)
 			(justify left)
+		)
+	)
+	(hierarchical_label "MISO_Master"
+		(shape output)
+		(at 179.07 109.22 0)
+		(effects
+			(font
+				(size 1.27 1.27)
+			)
+			(justify left)
+		)
+	)
+	(hierarchical_label "MISO_Slave"
+		(shape input)
+		(at 168.91 109.22 180)
+		(effects
+			(font
+				(size 1.27 1.27)
+			)
+			(justify right)
 		)
 	)
@@
 		(shape input)
 		(at 168.91 91.44 180)
-		(fields_autoplaced yes)
 		(effects
 			(font
@@
 		(on_board yes)
 		(dnp no)
-		(property "Reference" "R50"
+		(property "Reference" "R129"
 			(at 113.03 87.376 90)
 			(effects
@@
 			)
 		)
-		(property "Value" "4.7k"
+		(property "Value" "4k7"
 			(at 113.03 89.408 90)
 			(effects
@@
 			(project "Avionics-MainBoard"
 				(path "/4c932743-8c6f-426e-9c1f-5a3f2b32c70d/00f4ddfb-afd6-4184-9f71-0fb73daba661/61a7db01-d968-488e-83c5-60e79a23a452"
-					(reference "R50")
+					(reference "R129")
+					(unit 1)
+				)
+				(path "/4c932743-8c6f-426e-9c1f-5a3f2b32c70d/0c04e6a7-6d16-45e0-b82f-bf6f349905a8/dca4c2dc-4d01-4762-8a5d-b12bf5c24ee5"
+					(reference "R123")
 					(unit 1)
 				)
 				(path "/4c932743-8c6f-426e-9c1f-5a3f2b32c70d/6167394f-ef17-4174-a137-33bfda5b3a14/d6a2d62f-d8aa-4fe6-99dd-eb6ce237aeb0"
-					(reference "R57")
+					(reference "R107")
+					(unit 1)
+				)
+			)
+		)
+	)
+	(symbol
+		(lib_id "Device:R_Small")
+		(at 173.99 109.22 270)
+		(unit 1)
+		(exclude_from_sim no)
+		(in_bom yes)
+		(on_board yes)
+		(dnp yes)
+		(property "Reference" "R133"
+			(at 173.99 105.41 90)
+			(effects
+				(font
+					(size 1.27 1.27)
+				)
+			)
+		)
+		(property "Value" "0R"
+			(at 173.99 107.188 90)
+			(effects
+				(font
+					(size 1.27 1.27)
+				)
+			)
+		)
+		(property "Footprint" "Resistor_SMD:R_0603_1608Metric"
+			(at 173.99 109.22 0)
+			(effects
+				(font
+					(size 1.27 1.27)
+				)
+				(hide yes)
+			)
+		)
+		(property "Datasheet" "~"
+			(at 173.99 109.22 0)
+			(effects
+				(font
+					(size 1.27 1.27)
+				)
+				(hide yes)
+			)
+		)
+		(property "Description" "Resistor, small symbol"
+			(at 173.99 109.22 0)
+			(effects
+				(font
+					(size 1.27 1.27)
+				)
+				(hide yes)
+			)
+		)
+		(pin "1"
+		)
+		(pin "2"
+		)
+		(instances
+			(project "Avionics-MainBoard"
+				(path "/4c932743-8c6f-426e-9c1f-5a3f2b32c70d/00f4ddfb-afd6-4184-9f71-0fb73daba661/61a7db01-d968-488e-83c5-60e79a23a452"
+					(reference "R133")
+					(unit 1)
+				)
+				(path "/4c932743-8c6f-426e-9c1f-5a3f2b32c70d/0c04e6a7-6d16-45e0-b82f-bf6f349905a8/dca4c2dc-4d01-4762-8a5d-b12bf5c24ee5"
+					(reference "R127")
+					(unit 1)
+				)
+				(path "/4c932743-8c6f-426e-9c1f-5a3f2b32c70d/6167394f-ef17-4174-a137-33bfda5b3a14/d6a2d62f-d8aa-4fe6-99dd-eb6ce237aeb0"
+					(reference "R111")
 					(unit 1)
 				)
@@
 		(dnp no)
 		(fields_autoplaced yes)
-		(property "Reference" "Q14"
+		(property "Reference" "Q18"
 			(at 120.65 104.14 90)
 			(effects
@@
 			(project "Avionics-MainBoard"
 				(path "/4c932743-8c6f-426e-9c1f-5a3f2b32c70d/00f4ddfb-afd6-4184-9f71-0fb73daba661/61a7db01-d968-488e-83c5-60e79a23a452"
-					(reference "Q14")
+					(reference "Q18")
+					(unit 1)
+				)
+				(path "/4c932743-8c6f-426e-9c1f-5a3f2b32c70d/0c04e6a7-6d16-45e0-b82f-bf6f349905a8/dca4c2dc-4d01-4762-8a5d-b12bf5c24ee5"
+					(reference "Q17")
 					(unit 1)
 				)
 				(path "/4c932743-8c6f-426e-9c1f-5a3f2b32c70d/6167394f-ef17-4174-a137-33bfda5b3a14/d6a2d62f-d8aa-4fe6-99dd-eb6ce237aeb0"
-					(reference "Q15")
+					(reference "Q16")
 					(unit 1)
 				)
@@
 		(on_board yes)
 		(dnp no)
-		(property "Reference" "R52"
+		(property "Reference" "R132"
 			(at 173.99 96.266 90)
 			(effects
@@
 			(project "Avionics-MainBoard"
 				(path "/4c932743-8c6f-426e-9c1f-5a3f2b32c70d/00f4ddfb-afd6-4184-9f71-0fb73daba661/61a7db01-d968-488e-83c5-60e79a23a452"
-					(reference "R52")
+					(reference "R132")
+					(unit 1)
+				)
+				(path "/4c932743-8c6f-426e-9c1f-5a3f2b32c70d/0c04e6a7-6d16-45e0-b82f-bf6f349905a8/dca4c2dc-4d01-4762-8a5d-b12bf5c24ee5"
+					(reference "R126")
 					(unit 1)
 				)
 				(path "/4c932743-8c6f-426e-9c1f-5a3f2b32c70d/6167394f-ef17-4174-a137-33bfda5b3a14/d6a2d62f-d8aa-4fe6-99dd-eb6ce237aeb0"
-					(reference "R59")
+					(reference "R110")
 					(unit 1)
 				)
@@
 		(on_board yes)
 		(dnp no)
-		(property "Reference" "R51"
+		(property "Reference" "R131"
 			(at 173.99 87.376 90)
 			(effects
@@
 			(project "Avionics-MainBoard"
 				(path "/4c932743-8c6f-426e-9c1f-5a3f2b32c70d/00f4ddfb-afd6-4184-9f71-0fb73daba661/61a7db01-d968-488e-83c5-60e79a23a452"
-					(reference "R51")
+					(reference "R131")
+					(unit 1)
+				)
+				(path "/4c932743-8c6f-426e-9c1f-5a3f2b32c70d/0c04e6a7-6d16-45e0-b82f-bf6f349905a8/dca4c2dc-4d01-4762-8a5d-b12bf5c24ee5"
+					(reference "R125")
 					(unit 1)
 				)
 				(path "/4c932743-8c6f-426e-9c1f-5a3f2b32c70d/6167394f-ef17-4174-a137-33bfda5b3a14/d6a2d62f-d8aa-4fe6-99dd-eb6ce237aeb0"
-					(reference "R58")
+					(reference "R109")
 					(unit 1)
 				)
@@
 		(on_board yes)
 		(dnp no)
-		(property "Reference" "R49"
+		(property "Reference" "R130"
 			(at 110.49 96.52 90)
 			(effects
@@
 			(project "Avionics-MainBoard"
 				(path "/4c932743-8c6f-426e-9c1f-5a3f2b32c70d/00f4ddfb-afd6-4184-9f71-0fb73daba661/61a7db01-d968-488e-83c5-60e79a23a452"
-					(reference "R49")
+					(reference "R130")
+					(unit 1)
+				)
+				(path "/4c932743-8c6f-426e-9c1f-5a3f2b32c70d/0c04e6a7-6d16-45e0-b82f-bf6f349905a8/dca4c2dc-4d01-4762-8a5d-b12bf5c24ee5"
+					(reference "R124")
 					(unit 1)
 				)
 				(path "/4c932743-8c6f-426e-9c1f-5a3f2b32c70d/6167394f-ef17-4174-a137-33bfda5b3a14/d6a2d62f-d8aa-4fe6-99dd-eb6ce237aeb0"
-					(reference "R56")
-					(unit 1)
-				)
+					(reference "R108")
+					(unit 1)
+				)

Commit message: v4.0 Updates
Parts:
- renumbered R129 to R119, R130 to R120, R131 to R121, R132 to R122, R133 to R123
Changed lines of the file:
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@@
 (kicad_sch
-	(version 20231120)
+	(version 20250114)
 	(generator "eeschema")
-	(generator_version "8.0")
+	(generator_version "9.0")
 	(paper "A4")
 	(title_block
@@
 		(on_board yes)
 		(dnp no)
-		(property "Reference" "R129"
+		(property "Reference" "R119"
 			(at 113.03 87.376 90)
 			(effects
@@
 			(project "Avionics-MainBoard"
 				(path "/4c932743-8c6f-426e-9c1f-5a3f2b32c70d/00f4ddfb-afd6-4184-9f71-0fb73daba661/61a7db01-d968-488e-83c5-60e79a23a452"
-					(reference "R129")
-					(unit 1)
-				)
-				(path "/4c932743-8c6f-426e-9c1f-5a3f2b32c70d/0c04e6a7-6d16-45e0-b82f-bf6f349905a8/dca4c2dc-4d01-4762-8a5d-b12bf5c24ee5"
-					(reference "R123")
+					(reference "R119")
 					(unit 1)
 				)
@@
 		(on_board yes)
 		(dnp yes)
-		(property "Reference" "R133"
+		(property "Reference" "R123"
 			(at 173.99 105.41 90)
 			(effects
@@
 			(project "Avionics-MainBoard"
 				(path "/4c932743-8c6f-426e-9c1f-5a3f2b32c70d/00f4ddfb-afd6-4184-9f71-0fb73daba661/61a7db01-d968-488e-83c5-60e79a23a452"
-					(reference "R133")
-					(unit 1)
-				)
-				(path "/4c932743-8c6f-426e-9c1f-5a3f2b32c70d/0c04e6a7-6d16-45e0-b82f-bf6f349905a8/dca4c2dc-4d01-4762-8a5d-b12bf5c24ee5"
-					(reference "R127")
+					(reference "R123")
 					(unit 1)
 				)
@@
 					(unit 1)
 				)
-				(path "/4c932743-8c6f-426e-9c1f-5a3f2b32c70d/0c04e6a7-6d16-45e0-b82f-bf6f349905a8/dca4c2dc-4d01-4762-8a5d-b12bf5c24ee5"
+				(path "/4c932743-8c6f-426e-9c1f-5a3f2b32c70d/6167394f-ef17-4174-a137-33bfda5b3a14/d6a2d62f-d8aa-4fe6-99dd-eb6ce237aeb0"
 					(reference "Q17")
-					(unit 1)
-				)
-				(path "/4c932743-8c6f-426e-9c1f-5a3f2b32c70d/6167394f-ef17-4174-a137-33bfda5b3a14/d6a2d62f-d8aa-4fe6-99dd-eb6ce237aeb0"
-					(reference "Q16")
 					(unit 1)
 				)
@@
 		(on_board yes)
 		(dnp no)
-		(property "Reference" "R132"
+		(property "Reference" "R122"
 			(at 173.99 96.266 90)
 			(effects
@@
 			(project "Avionics-MainBoard"
 				(path "/4c932743-8c6f-426e-9c1f-5a3f2b32c70d/00f4ddfb-afd6-4184-9f71-0fb73daba661/61a7db01-d968-488e-83c5-60e79a23a452"
-					(reference "R132")
-					(unit 1)
-				)
-				(path "/4c932743-8c6f-426e-9c1f-5a3f2b32c70d/0c04e6a7-6d16-45e0-b82f-bf6f349905a8/dca4c2dc-4d01-4762-8a5d-b12bf5c24ee5"
-					(reference "R126")
+					(reference "R122")
 					(unit 1)
 				)
@@
 		(on_board yes)
 		(dnp no)
-		(property "Reference" "R131"
+		(property "Reference" "R121"
 			(at 173.99 87.376 90)
 			(effects
@@
 			(project "Avionics-MainBoard"
 				(path "/4c932743-8c6f-426e-9c1f-5a3f2b32c70d/00f4ddfb-afd6-4184-9f71-0fb73daba661/61a7db01-d968-488e-83c5-60e79a23a452"
-					(reference "R131")
-					(unit 1)
-				)
-				(path "/4c932743-8c6f-426e-9c1f-5a3f2b32c70d/0c04e6a7-6d16-45e0-b82f-bf6f349905a8/dca4c2dc-4d01-4762-8a5d-b12bf5c24ee5"
-					(reference "R125")
+					(reference "R121")
 					(unit 1)
 				)
@@
 		(on_board yes)
 		(dnp no)
-		(property "Reference" "R130"
+		(property "Reference" "R120"
 			(at 110.49 96.52 90)
 			(effects
@@
 			(project "Avionics-MainBoard"
 				(path "/4c932743-8c6f-426e-9c1f-5a3f2b32c70d/00f4ddfb-afd6-4184-9f71-0fb73daba661/61a7db01-d968-488e-83c5-60e79a23a452"
-					(reference "R130")
-					(unit 1)
-				)
-				(path "/4c932743-8c6f-426e-9c1f-5a3f2b32c70d/0c04e6a7-6d16-45e0-b82f-bf6f349905a8/dca4c2dc-4d01-4762-8a5d-b12bf5c24ee5"
-					(reference "R124")
-					(unit 1)
-				)
+					(reference "R120")
+					(unit 1)
+				)

Commit message: DFM updates
Parts:
- Q18: MPN (none) -> C5354954
- R119: MPN (none) -> C844931
- R120: MPN (none) -> C844915
- R121, R122: MPN (none) -> C2484712
- R123: DNI (none) -> DNI; now left out of the parts list
Changed lines of the file:
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@@
+			)
+		)
+		(property "MPN" "C844931"
+			(at 113.03 91.44 90)
+			(effects
+				(font
+					(size 1.27 1.27)
+				)
+				(hide yes)
 			)
 		)
@@
 		(unit 1)
 		(exclude_from_sim no)
-		(in_bom yes)
+		(in_bom no)
 		(on_board yes)
 		(dnp yes)
@@
 		(property "Description" "Resistor, small symbol"
 			(at 173.99 109.22 0)
+			(effects
+				(font
+					(size 1.27 1.27)
+				)
+				(hide yes)
+			)
+		)
+		(property "DNI" "DNI"
+			(at 173.99 109.22 90)
 			(effects
 				(font
@@
 			)
 		)
-		(property "Datasheet" "https://diotec.com/request/datasheet/mmbta56.pdf"
+		(property "Datasheet" ""
 			(at 120.65 97.79 0)
 			(effects
@@
 			)
 		)
-		(property "Flight" ""
-			(at 120.65 97.79 0)
-			(effects
-				(font
-					(size 1.27 1.27)
-				)
-				(hide yes)
-			)
-		)
-		(property "Manufacturer_Name" ""
+		(property "MPN" "C5354954"
 			(at 120.65 97.79 0)
 			(effects
@@
 			)
 		)
+		(property "MPN" "C2484712"
+			(at 173.99 100.33 90)
+			(effects
+				(font
+					(size 1.27 1.27)
+				)
+				(hide yes)
+			)
+		)
 		(pin "1"
 		)
@@
 			)
 		)
+		(property "MPN" "C2484712"
+			(at 173.99 91.44 90)
+			(effects
+				(font
+					(size 1.27 1.27)
+				)
+				(hide yes)
+			)
+		)
 		(pin "1"
 		)
@@
 			(effects
 				(font
+					(size 1.27 1.27)
+				)
+				(hide yes)
+			)
+		)
+		(property "MPN" "C844915"
+			(at 110.49 100.33 90)
+			(effects
+				(font
