File: SPI_Protection.kicad_sch (KiCad schematic)
At the start: 6 parts, among them Q18 MMBT2907

Commit message: v5.0 Updates
Parts:
- renumbered Q18 to Q24, R119 to R164, R120 to R165, R121 to R166, R122 to R167, R123 to R168
