File: USB.kicad_sch (KiCad schematic)
At the start: 21 parts, among them J1 USB_C_Receptacle_USB2.0, J3 Conn_01x06, U6 USBLC6-2SC6, U9 BQ25883RGER

Commit message: v1 done
Parts:
- J1: footprint Connector_USB:USB_C_Receptacle_HRO_TYPE-C-31-M-12 -> Connector_USB:USB_C_Receptacle_GCT_USB4105-xx-A_16P_TopMnt_Horizontal
- R46, R47: value 5.1K -> 5k1
- R65: value 5.23K -> 5k23
- R66: value 30.1K -> 30k1
- U9: symbol Mainboard:BQ25883RGER -> Argus-IC:BQ25883RGER
Connections:
- net D_UP+: now reaches J1.A6 (D+), J1.B6 (D+), U6.3 (I/O2)
- net D_UP-: now reaches J1.A7 (D-), J1.B7 (D-), U6.1 (I/O1)
Changed lines of the file:
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@@
+		)
+	)
+	(label "D_UP-"
+		(at 95.25 163.83 0)
+		(fields_autoplaced yes)
+		(effects
+			(font
+				(size 1.27 1.27)
+			)
+			(justify left bottom)
 		)
 	)
@@
 	(label "SYS"
 		(at 128.27 59.69 0)
+		(fields_autoplaced yes)
+		(effects
+			(font
+				(size 1.27 1.27)
+			)
+			(justify left bottom)
+		)
+	)
+	(label "D_UP+"
+		(at 95.25 166.37 0)
 		(fields_autoplaced yes)
 		(effects
@@
 			)
 		)
-		(property "Value" "5.1K"
+		(property "Value" "5k1"
 			(at 91.44 144.018 90)
 			(effects
@@
 			)
 		)
-		(property "Value" "30.1K"
+		(property "Value" "30k1"
 			(at 74.93 87.376 0)
 			(effects
@@
 			)
 		)
-		(property "Value" "5.1K"
+		(property "Value" "5k1"
 			(at 91.44 152.654 90)
 			(effects
@@
 			)
 		)
-		(property "Value" "5.23K"
+		(property "Value" "5k23"
 			(at 74.4982 78.613 0)
 			(effects
@@
 			)
 		)
-		(property "Footprint" "Connector_USB:USB_C_Receptacle_HRO_TYPE-C-31-M-12"
+		(property "Footprint" "Connector_USB:USB_C_Receptacle_GCT_USB4105-xx-A_16P_TopMnt_Horizontal"
 			(at 71.12 156.21 0)
 			(effects
@@
 	)
 	(symbol
-		(lib_id "Mainboard:BQ25883RGER")
+		(lib_id "Argus-IC:BQ25883RGER")
 		(at 82.55 54.61 0)
 		(unit 1)

Commit message: Updated version to v2.1
Other:
- company: (none) -> Carnegie Mellon University
- title: (none) -> Argus Mainboard
Changed lines of the file:
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@@
 	(generator_version "8.0")
 	(paper "A4")
+	(title_block
+		(title "Argus Mainboard")
+		(date "2024-11-19")
+		(rev "v2.1")
+		(company "Carnegie Mellon University")
+		(comment 1 "M. Holliday")
+		(comment 2 "N. Khera")
+		(comment 3 "V. Rajesh")
+	)
 	(junction
 		(at 113.03 59.69)

Commit message: v3 partial schematic updates
Parts:
- removed C38: 4u7, Capacitor_SMD:C_0603_1608Metric, symbol Device:C_Small
- removed D3: GREEN LED, LED_SMD:LED_0603_1608Metric, symbol Device:LED
- added C2: 4u7, Capacitor_SMD:C_0603_1608Metric, symbol Device:C_Small
- added D2: LED_G_0603_LTST-C190GKT, LED_SMD:LED_0603_1608Metric, symbol Device:LED_Small_Filled
- added R25: 0R, Resistor_SMD:R_0603_1608Metric, symbol Device:R_Small
- added R26: 1k91, Resistor_SMD:R_0603_1608Metric, symbol Device:R_Small
- J1: value USB_C_Receptacle_USB2.0 -> USB4105-GF-A
- L1: footprint Inductor_SMD:L_Wuerth_MAPI-2510 -> (none); Flight DFE252012F-1R0M -> DFE252012F-1R0M=P2; Manufacturer_Name Prosperity Dielectrics -> (none); Manufacturer_Part_Number MCS25GD-1R0MMP -> DFE252012F-1R0M=P2; Proto MCS25GD-1R0MMP -> DFE252012F-1R0M=P2
- R67, R70: value 10K -> 10k
- U9: value BQ25883RGER -> BQ25886RGER; symbol Argus-IC:BQ25883RGER -> Argus-IC:BQ25886RGER; Flight BQ25883RGER -> BQ25886RGER; Manufacturer_Part_Number BQ25883RGER -> BQ25886RGER; Proto BQ25883RGER -> BQ25886RGER
Connections:
- net CHG_SCL is gone; now on net GNDREF: U9.5 (OTG)
- net CHG_SDA is gone; now on net GNDREF: U9.4 (GND)
- net GNDREF: now also C2.2, R25.1, R26.2
- net REGN: now also C2.1
- net STAT: now also D2.1 (K)
- net at R70.1: now also D2.2 (A)
- net at U9.10 (ICHGSET): now also R26.1
- net at U9.6 (VSET): now also R25.2
- no-connect marks 6 -> 4
Other:
- removed sheet I2C Protection6
- note added: ""GND""
- note added: ""VBATT""
- note added: ""VSYS""
- note added: "Add VBATT jumper to allow USB battery charging (even inside P-Pod)."
- note added: "Add VSYS jumper to allow USB to power the board (even inside P-Pod)."
- note added: "Charge Current Limit Charge current (ICHG)=RICHGSET/KICHGSET KICHGSET = 3810 IINMAX = 500mA = 1.91 kohm"
- note added: "DNP R25 to charge to 8.4V Charges to 8.2V by default"
- note added: "Input Current Limit Max input current (IINMAX)=KILIM/RILIM KILIM = 1098 to 1276 at most IINMAX = 400mA = 3.16 kohm"
- note added: "RBF Jumpers"
- note added: "Remove both jumpers before flight to remove risk of unknown BQ25883 radiation failure modes"
- note added: "TODO: add note back in on disconnect jumpers"
- note added: "USB Connector"
- note removed: "0x6B"
- note removed: "I2C1 ADDR"
- note removed: "Input Current Limit Max input current (IINMAX)=KILIM/RILIM KILIM = 1098 to 1276 at most IINMAX=400mA=3.16 kohm"
- note removed: "add note back in on disconnect jumpers"
- moved on the sheet: C29, C37, C39, C40, C41, C42, C43, J1, J3, L1, R46, R47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

Commit message: v3 Layout complete
Parts:
- C23: renamed from C29; footprint Capacitor_SMD:C_0603_1608Metric -> Capacitor_SMD:C_0805_2012Metric
- C25: renamed from C39; footprint Capacitor_SMD:C_0603_1608Metric -> Capacitor_SMD:C_0805_2012Metric
- C26: renamed from C40; footprint Capacitor_SMD:C_0603_1608Metric -> Capacitor_SMD:C_1210_3225Metric
- C27: renamed from C42; footprint Capacitor_SMD:C_0603_1608Metric -> Capacitor_SMD:C_1210_3225Metric
- C29: renamed from C43; footprint Capacitor_SMD:C_0603_1608Metric -> Capacitor_SMD:C_0805_2012Metric
- C30: renamed from C2; footprint Capacitor_SMD:C_0603_1608Metric -> Capacitor_SMD:C_0805_2012Metric
- J2: renamed from J3; footprint Connector_PinHeader_2.54mm:PinHeader_1x06_P2.54mm_Vertical -> Connector_PinHeader_2.54mm:PinHeader_1x06_P2.54mm_Horizontal
- L1: footprint (none) -> Inductor_SMD:L_1008_2520Metric
- R17: renamed from R69; value 3.16K -> 3k16
- renumbered C37 to C24, C41 to C28, U6 to D1, R46 to R11, R47 to R12, R25 to R13, R65 to R14, R66 to R15, R67 to R16, R26 to R18, R70 to R19, U9 to U4
Connections:
- net BATT: now also J2.3 (Pin_3); no longer J2.5 (Pin_5)
- net D_UP+: now also D1.6 (I/O1); no longer D1.3 (I/O2)
- net D_UP-: now also D1.4 (I/O2); no longer D1.1 (I/O1)
- net GND: now also J2.5 (Pin_5); no longer J2.1 (Pin_1)
- net GNDREF: now also J2.6 (Pin_6); no longer J2.2 (Pin_2)
- net SYS: now also J2.1 (Pin_1); no longer J2.3 (Pin_3)
- net USB_D+: now also D1.1 (I/O1); no longer D1.4 (I/O2)
- net USB_D-: now also D1.3 (I/O2); no longer D1.6 (I/O1)
- net VBATT: now also J2.4 (Pin_4); no longer J2.6 (Pin_6)
- net VSYS: now also J2.2 (Pin_2); no longer J2.4 (Pin_4)
Other:
- moved on the sheet: J2

Commit message: Addressed design issues
Other:
- note added: "DNP R13 to charge to 8.4V Charges to 8.2V by default"
- note removed: "DNP R25 to charge to 8.4V Charges to 8.2V by default"
- note removed: "TODO: add note back in on disconnect jumpers"
Changed lines of the file:
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@@
-		)
-	)
-	(text "TODO: add note back in on disconnect jumpers"
-		(exclude_from_sim no)
-		(at 83.566 169.672 0)
-		(effects
-			(font
-				(size 2.54 2.54)
-			)
 		)
 	)
@@
 		)
 	)
-	(text "DNP R25 to charge to 8.4V\nCharges to 8.2V by default"
+	(text "DNP R13 to charge to 8.4V\nCharges to 8.2V by default"
 		(exclude_from_sim no)
 		(at 164.084 93.98 0)

Commit message: v4.0 Updates
Parts:
- removed C24: 1u, Capacitor_SMD:C_0603_1608Metric, symbol Device:C_Small
- removed C30: 4u7, Capacitor_SMD:C_0805_2012Metric, symbol Device:C_Small
- removed J2: Conn_01x06, Connector_PinHeader_2.54mm:PinHeader_1x06_P2.54mm_Horizontal, symbol Connector_Generic:Conn_01x06
- removed L1: 1uH, Inductor_SMD:L_1008_2520Metric, symbol Device:L
- removed R13: 0R, Resistor_SMD:R_0603_1608Metric, symbol Device:R_Small
- removed R14: 5k23, Resistor_SMD:R_0603_1608Metric, symbol Device:R_Small
- removed R15: 30k1, Resistor_SMD:R_0603_1608Metric, symbol Device:R_Small
- removed R16: 10k, Resistor_SMD:R_0603_1608Metric, symbol Device:R_Small
- removed R17: 3k16, Resistor_SMD:R_0603_1608Metric, symbol Device:R_Small
- removed R18: 1k91, Resistor_SMD:R_0603_1608Metric, symbol Device:R_Small
- removed U4: BQ25886RGER, Package_DFN_QFN:Texas_RGE0024H_VQFN-24-1EP_4x4mm_P0.5mm_EP2.7x2.7mm, symbol Argus-IC:BQ25886RGER
- added D3: DFLS130LQ-7, Diode_SMD:D_PowerDI-123, symbol Device:D_Schottky_Small
- added J2: 205338-0004, Connector_Molex:Molex_Pico-Lock_205338-0004_1x04-1MP_P2.00mm_Horizontal, symbol Connector_Generic_MountingPin:Conn_01x04_MountingPin
- added Q2: SIRA99DP-T1-GE3, Package_SO:PowerPAK_SO-8_Single, symbol Transistor_FET:Si7141DP
- added R19: 0R, Resistor_SMD:R_0603_1608Metric, symbol Device:R_Small
- added R20: 100k, Resistor_SMD:R_0603_1608Metric, symbol Device:R_Small
- added U4: LTC4412xS6, Package_TO_SOT_SMD:TSOT-23-6, symbol Power_Management:LTC4412xS6
- C25: value 10u -> 1u; footprint Capacitor_SMD:C_0805_2012Metric -> Capacitor_SMD:C_0603_1608Metric
- C28: value 47n -> 1u
- renumbered C29 to C24, D1 to D2, D2 to D4, R11 to R17, R12 to R18, R19 to R21
Connections:
- net BATT is gone; now on net VBATT: C24.2
- net REGN is gone; now on net VSYS: R21.2
- net STAT is gone; now on net GND: D4.1 (K)
- net SYS is gone; now on net VSYS: C26.2, C27.2
- net D_UP+: now also J2.2 (Pin_2)
- net D_UP-: now also J2.3 (Pin_3)
- net GND: now also C23.2, C24.1, C25.2, C26.1, C27.1, C28.2, D2.2 (GND), J1.A1 (GND), J1.A12 (GND), J1.B1 (GND), J1.B12 (GND), J1.S1 (SHIELD), R17.1, R18.1, J2.4 (Pin_4), J2.MP (MountPin), R20.2, U4.2 (GND), U4.3 (CTL)
- net VBATT: now also C25.1, Q2.5 (D), U4.1 (VIN)
- net VSYS: now also C28.1, D3.1 (K), Q2.1 (S), Q2.2 (S), Q2.3 (S), U4.6 (SENSE)
- net VUSB: now also D3.2 (A), R19.2, R20.1; no longer C23.1, D2.5 (VBUS), J1.A4 (VBUS), J1.A9 (VBUS), J1.B4 (VBUS), J1.B9 (VBUS)
- removed net GNDREF: C23.2, C24.1, C25.1, C26.1, C27.1, D2.2 (GND), J1.A1 (GND), J1.A12 (GND), J1.B1 (GND), J1.B12 (GND), J1.S1 (SHIELD), R17.1, R18.1
- new net: Q2.4 (G), U4.5 (GATE)
- new net VUSB_IN: C23.1, D2.5 (VBUS), J1.A4 (VBUS), J1.A9 (VBUS), J1.B4 (VBUS), J1.B9 (VBUS), J2.1 (Pin_1), R19.1
- no-connect marks 4 -> 3
Other:
- note removed: ""GND""
- note removed: ""VBATT""
- note removed: ""VSYS""
- note removed: "Add VBATT jumper to allow USB battery charging (even inside P-Pod)."
- note removed: "Add VSYS jumper to allow USB to power the board (even inside P-Pod)."
- note removed: "Charge Current Limit Charge current (ICHG)=RICHGSET/KICHGSET KICHGSET = 3810 IINMAX = 500mA = 1.91 kohm"
- note removed: "DNP R13 to charge to 8.4V Charges to 8.2V by default"
- note removed: "Input Current Limit Max input current (IINMAX)=KILIM/RILIM KILIM = 1098 to 1276 at most IINMAX = 400mA = 3.16 kohm"
- note removed: "RBF Jumpers"
- note removed: "Remove both jumpers before flight to remove risk of unknown BQ25883 radiation failure modes"
- note removed: "USB (Boost) Charging for 2-cell Li-Ion"
- moved on the sheet: C23, C24, C26, C27, D2, D4, J1, R17, R18, R21

Commit message: DFM updates
Parts:
- C23: MPN (none) -> C3861036
- C24: MPN (none) -> C386084
- C25, C28: MPN (none) -> C2214844
- C26, C27: MPN (none) -> C2803395
- D2: MPN (none) -> C7519
- D4: Author Antmicro -> (none); License Apache-2.0 -> (none); MPN LTST-C190GKT -> C2909774; Manufacturer Lite-On -> (none); Public False -> (none)
- J1: Flight U262-161N-4BVC11 -> (none); MPN (none) -> C3020560; Manufacturer_Name XKB Connectivity -> (none); Manufacturer_Part_Number U262-161N-4BVC11 -> (none); Proto U262-161N-4BVC11 -> (none)
- J2: MPN (none) -> C916325
- Q2: MPN (none) -> C3289459
- R17, R18: MPN (none) -> C2484686
- R19: MPN (none) -> C844915
- R20: MPN (none) -> C237792
- R21: MPN (none) -> C2479067
Changed lines of the file:
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@@
+			)
+		)
+		(property "MPN" "C2484686"
+			(at 73.66 85.09 90)
+			(effects
+				(font
+					(size 1.27 1.27)
+				)
+				(hide yes)
 			)
 		)
@@
 			)
 		)
+		(property "MPN" "C2484686"
+			(at 73.66 87.63 90)
+			(effects
+				(font
+					(size 1.27 1.27)
+				)
+				(hide yes)
+			)
+		)
 		(pin "1"
 		)
@@
 			)
 		)
+		(property "MPN" "C386084"
+			(at 182.88 106.68 0)
+			(effects
+				(font
+					(size 1.27 1.27)
+				)
+				(hide yes)
+			)
+		)
 		(pin "1"
 		)
@@
 			)
 		)
+		(property "MPN" "C2803395"
+			(at 227.33 99.06 0)
+			(effects
+				(font
+					(size 1.27 1.27)
+				)
+				(hide yes)
+			)
+		)
 		(pin "1"
 		)
@@
 			)
 		)
+		(property "MPN" "C237792"
+			(at 132.08 99.06 0)
+			(effects
+				(font
+					(size 1.27 1.27)
+				)
+				(hide yes)
+			)
+		)
 		(pin "1"
 		)
@@
 			)
 		)
-		(property "Flight" "U262-161N-4BVC11"
-			(at 49.53 95.25 0)
-			(effects
-				(font
-					(size 1.27 1.27)
-				)
-				(hide yes)
-			)
-		)
-		(property "Manufacturer_Name" "XKB Connectivity"
-			(at 52.2478 70.6882 0)
-			(effects
-				(font
-					(size 1.27 1.27)
-				)
-				(hide yes)
-			)
-		)
-		(property "Manufacturer_Part_Number" "U262-161N-4BVC11"
-			(at 52.2478 70.6882 0)
-			(effects
-				(font
-					(size 1.27 1.27)
-				)
-				(hide yes)
-			)
-		)
-		(property "Proto" "U262-161N-4BVC11"
+		(property "MPN" "C3020560"
 			(at 49.53 95.25 0)
 			(effects
@@
 			)
 		)
+		(property "MPN" "C2214844"
+			(at 190.5 106.68 0)
+			(effects
+				(font
+					(size 1.27 1.27)
+				)
+				(hide yes)
+			)
+		)
 		(pin "1"
 		)
@@
 		)
 		(property "Description" "22uF +-20% 10V X5R"
+			(at 236.22 99.06 0)
+			(effects
+				(font
+					(size 1.27 1.27)
+				)
+				(hide yes)
+			)
+		)
+		(property "MPN" "C2803395"
 			(at 236.22 99.06 0)
 			(effects
@@
 			)
 		)
+		(property "MPN" "C2479067"
+			(at 254 99.06 0)
+			(effects
+				(font
+					(size 1.27 1.27)
+				)
+				(hide yes)
+			)
+		)
 		(pin "1"
 		)
@@
 			)
 		)
+		(property "MPN" "C844915"
+			(at 124.46 80.01 90)
+			(effects
+				(font
+					(size 1.27 1.27)
+				)
+				(hide yes)
+			)
+		)
 		(pin "1"
 		)
@@
 		(property "Description" "-60A Id, -20V Vds, 1.9 mOhm Ron, PowerPAK-8"
 			(at 204.47 82.55 0)
+			(effects
+				(font
+					(size 1.27 1.27)
+				)
+				(hide yes)
+			)
+		)
+		(property "MPN" "C3289459"
+			(at 204.47 82.55 90)
 			(effects
 				(font
@@
 			)
 		)
+		(property "MPN" "C916325"
+			(at 41.91 142.24 0)
+			(effects
+				(font
+					(size 1.27 1.27)
+				)
+				(hide yes)
+			)
+		)
 		(pin "4"
 		)
@@
 			)
 		)
-		(property "MPN" "LTST-C190GKT"
+		(property "MPN" "C2909774"
 			(at 269.24 86.36 0)
 			(effects
@@
 			)
 		)
-		(property "Manufacturer" "Lite-On"
-			(at 271.78 86.36 0)
-			(effects
-				(font
-					(size 1.27 1.27)
-					(thickness 0.15)
-				)
-				(justify left bottom)
-				(hide yes)
-			)
-		)
-		(property "Author" "Antmicro"
-			(at 274.32 86.36 0)
-			(effects
-				(font
-					(size 1.27 1.27)
-					(thickness 0.15)
-				)
-				(justify left bottom)
-				(hide yes)
-			)
-		)
-		(property "License" "Apache-2.0"
-			(at 276.86 86.36 0)
-			(effects
-				(font
-					(size 1.27 1.27)
-					(thickness 0.15)
-				)
-				(justify left bottom)
-				(hide yes)
-			)
-		)
-		(property "Public" "False"
-			(at 271.78 88.9 0)
-			(effects
-				(font
-					(size 1.27 1.27)
-				)
-				(justify left bottom)
-				(hide yes)
-			)
-		)
 		(property "Color" "Green"
-			(at 255.524 110.49 90)
-			(effects
-				(font
-					(size 1.27 1.27)
-				)
-				(justify right)
-			)
-		)
-		(property "Sim.Pins" "1=K 2=A"
-			(at 254 109.22 0)
-			(effects
-				(font
-					(size 1.27 1.27)
-				)
-				(hide yes)
+			(at 258.318 110.49 90)
+			(effects
+				(font
+					(size 1.27 1.27)
+				)
 			)
 		)
@@
 			)
 		)
+		(property "MPN" "C7519"
+			(at 92.71 102.87 0)
+			(effects
+				(font
+					(size 1.27 1.27)
+				)
+				(hide yes)
+			)
+		)
 		(pin "5"
 		)
@@
 			)
 		)
+		(property "MPN" "C2214844"
+			(at 245.11 99.06 0)
+			(effects
+				(font
+					(size 1.27 1.27)
+				)
+				(hide yes)
+			)
+		)
 		(pin "1"
 		)
@@
 			(at 116.84 99.06 0)
 			(effects
+				(font
+					(size 1.27 1.27)
+				)
+				(hide yes)
+			)
+		)
+		(property "MPN" "C3861036"
+			(at 116.84 99.06 0)
+			(effects

Commit message: v4.2 Updates
Parts:
- removed C24: 10u, Capacitor_SMD:C_0805_2012Metric, symbol Device:C_Small
- removed C25: 1u, Capacitor_SMD:C_0603_1608Metric, symbol Device:C_Small
- removed D3: DFLS130LQ-7, Diode_SMD:D_PowerDI-123, symbol Device:D_Schottky_Small
- removed Q2: SIRA99DP-T1-GE3, Package_SO:PowerPAK_SO-8_Single, symbol Transistor_FET:Si7141DP
- removed U4: LTC4412xS6, Package_TO_SOT_SMD:TSOT-23-6, symbol Power_Management:LTC4412xS6
- added D15: LED_G_0603_LTST-C190GKT, LED_SMD:LED_0603_1608Metric, symbol Device:LED_Small_Filled
- added R150: 4k7, Resistor_SMD:R_0603_1608Metric, symbol Device:R_Small
Connections:
- net VSYS is gone; now on net VBATT: C26.2, C27.2, C28.1, R21.2
- net GND: now also D15.1 (K)
- net VUSB: now also R150.2
- new net: D15.2 (A), R150.1
- no-connect marks 3 -> 2
Other:
- moved on the sheet: C26, C27, C28, D4, R21
