File: WireProtection.kicad_sch (KiCad schematic)
At the start: 9 parts, among them Q4 NX3008NBKS, Q5 MBT2222ADW1T1

Commit message: temp
Parts:
- removed unit 2 of Q4
- removed unit 2 of Q5
- added Q2: MBT2222ADW1T1, Package_TO_SOT_SMD:SOT-363_SC-70-6, symbol Transistor_BJT:MBT2222ADW1T1
- added Q28: NX3008NBKS, Package_TO_SOT_SMD:SOT-363_SC-70-6, symbol BatteryBoard:NX3008NBKS
- renumbered C24 to C31, Q5 to Q12, Q4 to Q22, R100 to R102, R18 to R84, R19 to R85, R20 to R86, R21 to R87, R55 to R88
Connections:
- net BUS: now also Q2.3 (C2)
- net DEVICE: now also Q2.4 (E2)
- net GND: now also Q28.4 (S1)
- net at C31.1, R88.2: now also Q28.5 (G1)
- net at Q22.6 (D1), R84.2, R86.2: now also Q2.5 (B2)
- net at Q22.2 (G2), R85.2: now also Q28.3 (D2)

Commit message: v1 done
Parts:
- Q22: renamed from Q28; symbol BatteryBoard:NX3008NBKS -> Device:Q_Dual_NMOS_S1G1D2S2G2D1
- Q22: symbol BatteryBoard:NX3008NBKS -> Device:Q_Dual_NMOS_S1G1D2S2G2D1
- renumbered Q2 to Q12
Changed lines of the file:
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@@
 	(paper "A4")
 	(junction
-		(at 156.21 110.49)
+		(at 140.97 105.41)
 		(diameter 0)
 		(color 0 0 0 0)
@@
 	)
 	(junction
-		(at 140.97 105.41)
-		(diameter 0)
-		(color 0 0 0 0)
-	)
-	(junction
 		(at 146.05 80.01)
 		(diameter 0)
@@
 	(junction
 		(at 133.35 90.17)
+		(diameter 0)
+		(color 0 0 0 0)
+	)
+	(junction
+		(at 156.21 110.49)
 		(diameter 0)
 		(color 0 0 0 0)
@@
 	)
 	(symbol
-		(lib_id "BatteryBoard:NX3008NBKS")
-		(at 149.86 110.49 0)
+		(lib_id "Device:Q_Dual_NMOS_S1G1D2S2G2D1")
+		(at 151.13 110.49 0)
 		(mirror y)
 		(unit 2)
@@
 		(on_board yes)
 		(dnp no)
-		(property "Reference" "Q28"
-			(at 145.796 110.49 0)
+		(property "Reference" "Q22"
+			(at 147.066 110.49 0)
 			(effects
 				(font
@@
 		)
 		(property "Value" "NX3008NBKS"
-			(at 161.544 123.19 0)
+			(at 162.814 123.19 0)
 			(effects
 				(font
@@
 		)
 		(property "Footprint" "Package_TO_SOT_SMD:SOT-363_SC-70-6"
-			(at 163.83 124.46 0)
+			(at 146.05 110.49 0)
+			(effects
+				(font
+					(size 1.27 1.27)
+				)
+				(hide yes)
+			)
+		)
+		(property "Datasheet" "~"
+			(at 146.05 110.49 0)
+			(effects
+				(font
+					(size 1.27 1.27)
+				)
+				(hide yes)
+			)
+		)
+		(property "Description" "Dual NMOS transistor, 6 pin package"
+			(at 151.13 110.49 0)
+			(effects
+				(font
+					(size 1.27 1.27)
+				)
+				(hide yes)
+			)
+		)
+		(property "Manufacturer_Name" "Nexperia USA Inc."
+			(at 165.1 132.08 0)
 			(effects
 				(font
@@
 			)
 		)
-		(property "Datasheet" "https://assets.nexperia.com/documents/data-sheet/NX3008NBKS.pdf"
-			(at 163.83 127 0)
+		(property "Manufacturer_Part_Number" "NX3008NBKS"
+			(at 165.1 134.62 0)
 			(effects
 				(font
@@
 			)
 		)
-		(property "Description" "Dual N-Channel MOSFET - 2NMOS"
-			(at 163.83 129.54 0)
-			(effects
-				(font
-					(size 1.27 1.27)
-				)
-				(justify left)
-				(hide yes)
-			)
-		)
-		(property "Manufacturer_Name" "Nexperia USA Inc."
-			(at 163.83 132.08 0)
-			(effects
-				(font
-					(size 1.27 1.27)
-				)
-				(justify left)
-				(hide yes)
-			)
-		)
-		(property "Manufacturer_Part_Number" "NX3008NBKS"
-			(at 163.83 134.62 0)
-			(effects
-				(font
-					(size 1.27 1.27)
-				)
-				(justify left)
-				(hide yes)
-			)
-		)
 		(property "Proto" "BSS138DWQ-7"
-			(at 149.86 110.49 0)
+			(at 151.13 110.49 0)
 			(effects
 				(font
@@
 		(on_board yes)
 		(dnp no)
-		(property "Reference" "Q2"
+		(property "Reference" "Q12"
 			(at 151.13 83.439 90)
 			(effects
@@
 	)
 	(symbol
-		(lib_id "BatteryBoard:NX3008NBKS")
-		(at 134.62 105.41 0)
+		(lib_id "Device:Q_Dual_NMOS_S1G1D2S2G2D1")
+		(at 135.89 105.41 0)
 		(mirror y)
 		(unit 1)
@@
 		(dnp no)
 		(property "Reference" "Q22"
-			(at 130.556 105.41 0)
+			(at 131.826 105.41 0)
 			(effects
 				(font
@@
 		)
 		(property "Value" "NX3008NBKS"
-			(at 146.304 118.11 0)
+			(at 147.574 118.11 0)
 			(effects
 				(font
@@
 		)
 		(property "Footprint" "Package_TO_SOT_SMD:SOT-363_SC-70-6"
-			(at 148.59 119.38 0)
+			(at 130.81 105.41 0)
+			(effects
+				(font
+					(size 1.27 1.27)
+				)
+				(hide yes)
+			)
+		)
+		(property "Datasheet" "~"
+			(at 130.81 105.41 0)
+			(effects
+				(font
+					(size 1.27 1.27)
+				)
+				(hide yes)
+			)
+		)
+		(property "Description" "Dual NMOS transistor, 6 pin package"
+			(at 135.89 105.41 0)
+			(effects
+				(font
+					(size 1.27 1.27)
+				)
+				(hide yes)
+			)
+		)
+		(property "Manufacturer_Name" "Nexperia USA Inc."
+			(at 149.86 127 0)
 			(effects
 				(font
@@
 			)
 		)
-		(property "Datasheet" "https://assets.nexperia.com/documents/data-sheet/NX3008NBKS.pdf"
-			(at 148.59 121.92 0)
+		(property "Manufacturer_Part_Number" "NX3008NBKS"
+			(at 149.86 129.54 0)
 			(effects
 				(font
@@
 			)
 		)
-		(property "Description" "Dual N-Channel MOSFET - 2NMOS"
-			(at 148.59 124.46 0)
-			(effects
-				(font
-					(size 1.27 1.27)
-				)
-				(justify left)
-				(hide yes)
-			)
-		)
-		(property "Manufacturer_Name" "Nexperia USA Inc."
-			(at 148.59 127 0)
-			(effects
-				(font
-					(size 1.27 1.27)
-				)
-				(justify left)
-				(hide yes)
-			)
-		)
-		(property "Manufacturer_Part_Number" "NX3008NBKS"
-			(at 148.59 129.54 0)
-			(effects
-				(font
-					(size 1.27 1.27)
-				)
-				(justify left)
-				(hide yes)
-			)
-		)
 		(property "Proto" "BSS138DWQ-7"
-			(at 134.62 105.41 0)
-			(effects
-				(font
+			(at 135.89 105.41 0)
+			(effects
+				(font

Commit message: Updated version to v2.1
Other:
- company: (none) -> Carnegie Mellon University
- title: (none) -> Argus Mainboard
Changed lines of the file:
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@@
 	(generator_version "8.0")
 	(paper "A4")
+	(title_block
+		(title "Argus Mainboard")
+		(date "2024-11-19")
+		(rev "v2.1")
+		(company "Carnegie Mellon University")
+		(comment 1 "M. Holliday")
+		(comment 2 "N. Khera")
+		(comment 3 "V. Rajesh")
+	)
 	(junction
 		(at 140.97 105.41)

Commit message: v3 partial schematic updates
Parts:
- R103: renamed from R102; value DNI (0R) -> 0R; now not fitted
- R90: renamed from R85; value 100K -> 100k
- R91: renamed from R86; value 10K -> 10k
- R92: renamed from R87; value 10K -> 10k
- R93: renamed from R88; value 200K -> 200k
- renumbered C31 to C35, Q12 to Q13, Q22 to Q24, R84 to R89
Connections:
- net +3V3 renamed 3V3
Other:
- note added: "TODO: CHANGE 3V3"
- moved on the sheet: C35, Q13B, R89, R92, R93

Commit message: v3 Layout complete
Parts:
- renumbered C35 to C54, Q13 to Q4, Q24 to Q5, R91 to R54, R92 to R55, R89 to R56, R90 to R57, R93 to R58, R103 to R59
Other:
- note removed: "TODO: CHANGE 3V3"

Commit message: v4.0 Updates
Parts:
- renumbered C54 to C62, Q4 to Q13, Q5 to Q14, R59 to R100, R54 to R95, R55 to R96, R56 to R97, R57 to R98, R58 to R99

Commit message: DFM updates
Parts:
- C62: MPN (none) -> C161232
- Q14: MPN (none) -> C3280240; Manufacturer_Name Nexperia USA Inc. -> (none); Manufacturer_Part_Number NX3008NBKS -> (none); Proto BSS138DWQ-7 -> (none)
- R100: now left out of the parts list
- R95, R96: MPN (none) -> C2479067
- R97: MPN (none) -> C844802
- R98: MPN (none) -> C237792
- R99: MPN (none) -> C118142
Changed lines of the file:
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@@
 			)
 		)
-		(property "Manufacturer_Name" "Nexperia USA Inc."
+		(property "MPN" "C3280240"
 			(at 165.1 132.08 0)
 			(effects
@@
 				)
 				(justify left)
-				(hide yes)
-			)
-		)
-		(property "Manufacturer_Part_Number" "NX3008NBKS"
-			(at 165.1 134.62 0)
-			(effects
-				(font
-					(size 1.27 1.27)
-				)
-				(justify left)
-				(hide yes)
-			)
-		)
-		(property "Proto" "BSS138DWQ-7"
-			(at 151.13 110.49 0)
-			(effects
-				(font
-					(size 1.27 1.27)
-				)
 				(hide yes)
 			)
@@
 			)
 		)
+		(property "MPN" "C161232"
+			(at 157.48 114.3 0)
+			(effects
+				(font
+					(size 1.27 1.27)
+				)
+				(hide yes)
+			)
+		)
 		(pin "1"
 		)
@@
 			)
 		)
+		(property "MPN" "C237792"
+			(at 140.97 101.6 0)
+			(effects
+				(font
+					(size 1.27 1.27)
+				)
+				(hide yes)
+			)
+		)
 		(pin "1"
 		)
@@
 		(unit 1)
 		(exclude_from_sim no)
-		(in_bom yes)
+		(in_bom no)
 		(on_board yes)
 		(dnp yes)
@@
 			)
 		)
+		(property "MPN" "C118142"
+			(at 157.48 104.14 0)
+			(effects
+				(font
+					(size 1.27 1.27)
+				)
+				(hide yes)
+			)
+		)
 		(pin "1"
 		)
@@
 			)
 		)
+		(property "MPN" "C844802"
+			(at 139.7 88.9 90)
+			(effects
+				(font
+					(size 1.27 1.27)
+				)
+				(hide yes)
+			)
+		)
 		(pin "1"
 		)
@@
 		)
 		(property "Description" "Resistor, small symbol"
+			(at 151.13 68.58 0)
+			(effects
+				(font
+					(size 1.27 1.27)
+				)
+				(hide yes)
+			)
+		)
+		(property "MPN" "C2479067"
 			(at 151.13 68.58 0)
 			(effects
@@
 			)
 		)
-		(property "Manufacturer_Name" "Nexperia USA Inc."
+		(property "MPN" "C3280240"
 			(at 149.86 127 0)
 			(effects
@@
 				)
 				(justify left)
-				(hide yes)
-			)
-		)
-		(property "Manufacturer_Part_Number" "NX3008NBKS"
-			(at 149.86 129.54 0)
-			(effects
-				(font
-					(size 1.27 1.27)
-				)
-				(justify left)
-				(hide yes)
-			)
-		)
-		(property "Proto" "BSS138DWQ-7"
-			(at 135.89 105.41 0)
-			(effects
-				(font
-					(size 1.27 1.27)
-				)
 				(hide yes)
 			)
@@
 			(at 157.48 74.93 0)
 			(effects
+				(font
+					(size 1.27 1.27)
+				)
+				(hide yes)
+			)
+		)
+		(property "MPN" "C2479067"
+			(at 157.48 74.93 0)
+			(effects

Commit message: v4.2 Updates
Parts:
- Q14: symbol Device:Q_Dual_NMOS_S1G1D2S2G2D1 -> Transistor_FET:Q_Dual_NMOS_S1G1D2S2G2D1
Changed lines of the file:
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@@
 	(title_block
 		(title "Argus Mainboard")
-		(date "2025-01-08")
-		(rev "v3.0")
+		(date "2025-11-24")
+		(rev "v4.2")
 		(company "Carnegie Mellon University")
 		(comment 1 "M. Holliday")
@@
 	)
 	(symbol
-		(lib_id "Device:Q_Dual_NMOS_S1G1D2S2G2D1")
+		(lib_id "Transistor_FET:Q_Dual_NMOS_S1G1D2S2G2D1")
 		(at 151.13 110.49 0)
 		(mirror y)
@@
 	)
 	(symbol
-		(lib_id "Device:Q_Dual_NMOS_S1G1D2S2G2D1")
+		(lib_id "Transistor_FET:Q_Dual_NMOS_S1G1D2S2G2D1")
 		(at 135.89 105.41 0)
 		(mirror y)
