File: WireProtection.kicad_sch (KiCad schematic)
At the start: 9 parts, among them Q13 MBT2222ADW1T1, Q14 NX3008NBKS

Commit message: v5.0 Updates
Parts:
- Q4: renamed from Q13; footprint Package_TO_SOT_SMD:SOT-363_SC-70-6 -> Argus-IC:SOT-363_SC-70-6
- Q5: renamed from Q14; footprint Package_TO_SOT_SMD:SOT-363_SC-70-6 -> Argus-IC:SOT-363_SC-70-6
- renumbered C62 to C40, R95 to R36, R96 to R37, R97 to R38, R98 to R39, R99 to R40, R100 to R41
