File: SD.kicad_sch (KiCad schematic)
At the start: 5 parts, among them J4 104031-0811

Commit message: v5.0 Updates
Parts:
- removed F1: 500mA, Fuse:Fuse_0603_1608Metric, symbol Device:Fuse_Small
- added C69: 10u, Capacitor_SMD:C_0805_2012Metric, symbol Device:C_Small
- added C70: 1u, Capacitor_SMD:C_0603_1608Metric, symbol Device:C_Small
- added C71: 1n, Capacitor_SMD:C_0603_1608Metric, symbol Device:C_Small
- added C72: 22u, Capacitor_SMD:C_1210_3225Metric, symbol Device:C_Small
- added D15: LED_G_0603_LTST-C190GKT, LED_SMD:LED_0603_1608Metric, symbol Device:LED_Small_Filled
- added R126, R127, R128: 0R, Resistor_SMD:R_0603_1608Metric, symbol Device:R_Small
- added R129, R131: 100k, Resistor_SMD:R_0603_1608Metric, symbol Device:R_Small
- added R130: 2k7, Resistor_SMD:R_0603_1608Metric, symbol Device:R_Small
- added U16: TPS22992, Argus-IC:TPS22992, symbol Argus-IC:TPS22992
- C73: renamed from C70; value 47u -> 22u
- renumbered C71 to C74, J4 to J13, R118 to R132
Connections:
- net +3V3_P: now also R126.1
- net +3V3_SD: now also C72.1, R128.1, R129.1, R130.2, U16.6 (VOUT)
- net GND: now also J13.SH (SHIELD), C69.2, C70.2, C71.2, C72.2, D15.1 (K), R131.2, U16.4 (GND); no longer J13.11 (SHIELD)
- new net: C69.1, C70.1, R126.2, R127.2, R128.2, U16.1 (VBIAS), U16.2 (VIN)
- new net: D15.2 (A), R130.1
- new net: R129.2, U16.5 (QOD)
- new net: C71.1, U16.7 (CT)
- new net +3V3_M: R127.1
- new net SD_EN: R131.1, U16.8 (ON)
- no-connect marks 4 -> 5
Other:
- note added: "MicroSD Enable"
- note added: "Slew rate for C71 = 1000pF = 962 us Use >= 50V cap"
- moved on the sheet: C73, C74, J13, R132
