File: SD.kicad_sch (KiCad schematic)
At the start: 16 parts, among them J13 104031-0811, U16 TPS22992

Commit message: Final v5.0 Release
Connections:
- net at D15.2 (A), R130.1: now also U16.3 (PG)
- no-connect marks 5 -> 4
Changed lines of the file:
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@@
+	)
+	(junction
+		(at 127 85.725)
+		(diameter 0)
+		(color 0 0 0 0)
 	)
 	(junction
@@
 		(at 190.5 98.425)
 	)
-	(no_connect
-		(at 107.315 88.9)
+	(wire
+		(pts
+			(xy 107.315 88.9) (xy 121.92 88.9)
+		)
+		(stroke
+			(width 0)
+			(type default)
+		)
 	)
 	(wire
@@
 	(wire
 		(pts
+			(xy 127 85.725) (xy 127 86.36)
+		)
+		(stroke
+			(width 0)
+			(type default)
+		)
+	)
+	(wire
+		(pts
 			(xy 118.11 78.74) (xy 127 78.74)
 		)
@@
 	(wire
 		(pts
-			(xy 127 85.09) (xy 127 86.36)
+			(xy 127 85.09) (xy 127 85.725)
 		)
 		(stroke
@@
 	(wire
 		(pts
+			(xy 121.92 88.9) (xy 121.92 85.725)
+		)
+		(stroke
+			(width 0)
+			(type default)
+		)
+	)
+	(wire
+		(pts
 			(xy 71.755 107.315) (xy 71.755 106.045)
 		)
@@
 		)
 		(stroke
+			(width 0)
+			(type default)
+		)
+	)
+	(wire
+		(pts
+			(xy 121.92 85.725) (xy 127 85.725)
+		)
+		(stroke
