File: Connectors.kicad_sch (KiCad schematic)
At the start: 15 parts, among them J10 522711069, J11 522711069, J12 522711069, J13 522711069, J14 282834-2, J15 282834-2, J16 282834-2, J17 205338-0002, J18 205338-0002, J19 205338-0002, J5 522711069, J6 522711069, J7 522711069, J8 522711069, J9 522711069

Commit message: v5.0 Updates
Parts:
- removed J10, J11, J12, J13, J5, J6, J7, J8, J9: 522711069, Argus-Connectors:CON_522711069_MOL, symbol Connector_Generic_MountingPin:Conn_01x10_MountingPin
- removed J14, J15, J16: 282834-2, Argus-Connectors:TE_282834-2, symbol Connector_Generic:Conn_01x02
- removed J17, J18, J19: 205338-0002, Connector_Molex:Molex_Pico-Lock_205338-0002_1x02-1MP_P2.00mm_Horizontal, symbol Connector_Generic_MountingPin:Conn_01x02_MountingPin
- added H5, H6: MountingHole_Pad, MountingHole:MountingHole_2.7mm_M2.5_Pad_Via, symbol Mechanical:MountingHole_Pad
- added J14: QSH-030-01-L-D-A, Argus-Connectors:SAMTEC_QSH-030-01-L-D-A, symbol Connector_Generic_Shielded:Conn_02x30_Odd_Even_Shielded
- added J15: QTH-030-01-L-D-A, Argus-Connectors:SAMTEC-QTH-030-01-X-D-A, symbol Connector_Generic_Shielded:Conn_02x30_Odd_Even_Shielded
Connections:
- net +3V3_P: now also J14.21 (Pin_21), J14.22 (Pin_22), J14.23 (Pin_23), J14.24 (Pin_24), J15.21 (Pin_21), J15.22 (Pin_22), J15.23 (Pin_23), J15.24 (Pin_24)
- net GND: now also H5.1, H6.1, J14.11 (Pin_11), J14.12 (Pin_12), J14.13 (Pin_13), J14.14 (Pin_14), J14.15 (Pin_15), J14.16 (Pin_16), J14.17 (Pin_17), J14.18 (Pin_18), J14.19 (Pin_19), J14.20 (Pin_20), J14.25 (Pin_25), J14.26 (Pin_26), J14.27 (Pin_27), J14.28 (Pin_28), J14.35 (Pin_35), J14.41 (Pin_41), J14.44 (Pin_44), J14.45 (Pin_45), J14.59 (Pin_59), J14.60 (Pin_60), J14.SH (Shield), J15.11 (Pin_11), J15.12 (Pin_12), J15.13 (Pin_13), J15.14 (Pin_14), J15.15 (Pin_15), J15.16 (Pin_16), J15.17 (Pin_17), J15.18 (Pin_18), J15.19 (Pin_19), J15.20 (Pin_20), J15.25 (Pin_25), J15.26 (Pin_26), J15.27 (Pin_27), J15.28 (Pin_28), J15.35 (Pin_35), J15.41 (Pin_41), J15.44 (Pin_44), J15.45 (Pin_45), J15.59 (Pin_59), J15.60 (Pin_60), J15.SH (Shield)
- net I2C0_SCL: now also J14.37 (Pin_37), J15.37 (Pin_37)
- net I2C0_SDA: now also J14.39 (Pin_39), J15.39 (Pin_39)
- new net BUS_IO01: J14.30 (Pin_30), J15.30 (Pin_30)
- new net BUS_IO02: J14.32 (Pin_32), J15.32 (Pin_32)
- new net BUS_IO03: J14.34 (Pin_34), J15.34 (Pin_34)
- new net BUS_IO04: J14.36 (Pin_36), J15.36 (Pin_36)
- new net BUS_IO05: J14.38 (Pin_38), J15.38 (Pin_38)
- new net BUS_IO06: J14.40 (Pin_40), J15.40 (Pin_40)
- new net BUS_IO07: J14.42 (Pin_42), J15.42 (Pin_42)
- new net BUS_IO08: J14.46 (Pin_46), J15.46 (Pin_46)
- new net BUS_IO09: J14.48 (Pin_48), J15.48 (Pin_48)
- new net BUS_IO10: J14.50 (Pin_50), J15.50 (Pin_50)
- new net BUS_IO11: J14.52 (Pin_52), J15.52 (Pin_52)
- new net BUS_IO12: J14.54 (Pin_54), J15.54 (Pin_54)
- new net BUS_IO13: J14.56 (Pin_56), J15.56 (Pin_56)
- new net BUS_IO14: J14.58 (Pin_58), J15.58 (Pin_58)
- new net FREE_IO1: J14.47 (Pin_47), J15.47 (Pin_47)
- new net FREE_IO2: J14.49 (Pin_49), J15.49 (Pin_49)
- new net FREE_IO3: J14.51 (Pin_51), J15.51 (Pin_51)
- new net FREE_IO4: J14.53 (Pin_53), J15.53 (Pin_53)
- new net FREE_IO5: J14.55 (Pin_55), J15.55 (Pin_55)
- new net FREE_IO6: J14.57 (Pin_57), J15.57 (Pin_57)
- new net GPS_1PPS: J14.43 (Pin_43), J15.43 (Pin_43)
- new net SPI0_CLK: J14.29 (Pin_29), J15.29 (Pin_29)
- new net SPI0_MISO: J14.33 (Pin_33), J15.33 (Pin_33)
- new net SPI0_MOSI: J14.31 (Pin_31), J15.31 (Pin_31)
- new net VBATT: J14.1 (Pin_1), J14.10 (Pin_10), J14.2 (Pin_2), J14.3 (Pin_3), J14.4 (Pin_4), J14.5 (Pin_5), J14.6 (Pin_6), J14.7 (Pin_7), J14.8 (Pin_8), J14.9 (Pin_9), J15.1 (Pin_1), J15.10 (Pin_10), J15.2 (Pin_2), J15.3 (Pin_3), J15.4 (Pin_4), J15.5 (Pin_5), J15.6 (Pin_6), J15.7 (Pin_7), J15.8 (Pin_8), J15.9 (Pin_9)
Other:
- note added: "ADCS_CS"
- note added: "ADCS_EN"
- note added: "BATT0_EN"
- note added: "BATT1_EN"
- note added: "BATT_ALRT"
- note added: "BOTTOM"
- note added: "Payload_En"
- note added: "Payload_IO1"
- note added: "Payload_IO2"
- note added: "Payload_IO3"
- note added: "RW_EN"
- note added: "RW_MTR_ALRM"
- note added: "RW_MTR_FLT"
- note added: "RW_PWR_FLT"
- note added: "RW_SCL"
- note added: "RW_SDA"
- note added: "TODO: 0ohm"
- note added: "TOP"
- note added: "eGPS_EN"
- note added: "eGPS_RX"
- note added: "eGPS_TX"
- note removed: "+X"
- note removed: "+Y"
- note removed: "+Z"
- note removed: "-X"
- note removed: "-Y"
- note removed: "-Z"
- note removed: "BatteryBoard"
- note removed: "Jetson"
- note removed: "Power Out"
- note removed: "Reaction Wheel"
- note removed: "Solar Panel Connectors"

Commit message: Final v5.0 Release
Other:
- note removed: "TODO: 0ohm"
Changed lines of the file:
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@@
+		)
+	)
+	(text "RW_PWR_FLT"
+		(exclude_from_sim no)
+		(at 161.29 120.015 0)
+		(effects
+			(font
+				(size 1.27 1.27)
+			)
+			(justify right)
 		)
 	)
@@
 		)
 	)
+	(text "RW_MTR_FLT"
+		(exclude_from_sim no)
+		(at 161.29 122.555 0)
+		(effects
+			(font
+				(size 1.27 1.27)
+			)
+			(justify right)
+		)
+	)
 	(text "ADCS_CS"
 		(exclude_from_sim no)
@@
 		)
 	)
-	(text "TODO: 0ohm"
-		(exclude_from_sim no)
-		(at 155.575 112.395 0)
-		(effects
-			(font
-				(size 1.27 1.27)
-			)
+	(text "RW_MTR_ALRM"
+		(exclude_from_sim no)
+		(at 161.29 125.095 0)
+		(effects
+			(font
+				(size 1.27 1.27)
+			)
+			(justify right)
 		)
 	)
@@
 		)
 	)
+	(text "RW_EN"
+		(exclude_from_sim no)
+		(at 161.29 117.475 0)
+		(effects
+			(font
+				(size 1.27 1.27)
+			)
+			(justify right)
+		)
+	)
 	(text "Payload_IO3"
 		(exclude_from_sim no)
@@
 		)
 	)
+	(text "RW_SDA"
+		(exclude_from_sim no)
+		(at 161.29 130.175 0)
+		(effects
+			(font
+				(size 1.27 1.27)
+			)
+			(justify right)
+		)
+	)
 	(text "Payload_En"
 		(exclude_from_sim no)
@@
 		(effects
 			(font
+				(size 1.27 1.27)
+			)
+			(justify right)
+		)
+	)
+	(text "RW_SCL"
+		(exclude_from_sim no)
+		(at 161.29 127.635 0)
+		(effects
+			(font
