File: PowerSelection.kicad_sch (KiCad schematic)
At the start: 27 parts, among them J1 USB4105-GF-A, J10 282834-4, J2 205338-0004, J3 205338-0004, Q2 FDC6327C, Q3 DMP3056L, U5 LTC4412xS6

Commit message: Final v5.0 Release
Parts:
- Q2: value FDC6327C -> DMC3060LVT
Changed lines of the file:
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@@
 			)
 		)
-		(property "Value" "FDC6327C"
+		(property "Value" "DMC3060LVT"
 			(at 247.015 92.075 0)
 			(show_name no)
@@
 			)
 		)
-		(property "Value" "FDC6327C"
+		(property "Value" "DMC3060LVT"
 			(at 227.33 112.395 0)
 			(show_name no)
