File: RTC.kicad_sch (KiCad schematic)
At the start: 4 parts, among them U17 DS3231SN

Commit message: v5.0 Updates
Parts:
- removed F2: 50mA, Fuse:Fuse_0603_1608Metric, symbol Device:Fuse_Small
- removed U17: DS3231SN, Package_SO:SOIC-16W_7.5x10.3mm_P1.27mm, symbol Timer_RTC:DS3231M
- added C75, C76: 10u, Capacitor_SMD:C_0805_2012Metric, symbol Device:C_Small
- added C78: 100n, Capacitor_SMD:C_0603_1608Metric, symbol Device:C_Small
- added D16: LED_G_0603_LTST-C190GKT, LED_SMD:LED_0603_1608Metric, symbol Device:LED_Small_Filled
- added R138, R139, R140: 0R, Resistor_SMD:R_0603_1608Metric, symbol Device:R_Small
- added R141, R143, R144, R185: 10k, Resistor_SMD:R_0603_1608Metric, symbol Device:R_Small
- added R142: 2k7, Resistor_SMD:R_0603_1608Metric, symbol Device:R_Small
- added TP8: TestPoint, TestPoint:TestPoint_Pad_D1.5mm, symbol Connector:TestPoint
- added U17: TPS22917DBV, Package_TO_SOT_SMD:SOT-23-6, symbol Power_Management:TPS22917DBV
- added U18: RV-3032-C7, Argus-IC:IC_RV-3032-C7-32.768KHZ-2.5PPM-TA-QC, symbol Argus-IC:RV-3032-C7-32.768KHZ-2.5PPM-TA-QC
- BT2: renamed from BT1; value 3.0V -> BAT-HLD-012-SMT; Field6 (none) -> CR1225
- renumbered C72 to C77
Connections:
- net +3V3_P: now also R139.1
- net +3V3_RTC: now also C76.1, R140.1, R142.2, R143.1, R185.2, U17.6 (VOUT), U18.6 (VDD)
- net GND: now also C75.2, C76.2, C78.2, D16.1 (K), R141.2, R144.2, U17.2 (GND), U18.5 (VSS)
- net RTC_SCL: now also U18.8 (SCL)
- net RTC_SDA: now also U18.2 (SDA)
- net at BT2.1 (+): now also C78.1, U18.1 (VBACKUP)
- new net: TP8.1, U18.7 (CLKOUT)
- new net: C75.1, R138.2, R139.2, R140.2, U17.1 (VIN)
- new net: R185.1, U17.5 (QOD)
- new net: D16.2 (A), R142.1
- new net +3V3_M: R138.1
- new net EVI: R144.1, U18.4 (EVI)
- new net RTC_EN: R141.1, U17.3 (ON)
- new net RTC_INT: R143.2, U18.3 (~{INT})
- no-connect marks 3 -> 1
Other:
- note added: "I2C1 ADDR 0x51"
- note added: "RTC"
- note added: "RTC Enable"
- note removed: "I2C1 ADDR 0x68"
- note removed: "TODO: Add some way to do full component power cycle"
- moved on the sheet: BT2, C77

Commit message: Final v5.0 Release
Parts:
- R141, R144: value 10k -> 100k
- TP8: now left out of the parts list
Connections:
- net +3V3_M: now also R143.1
- net +3V3_RTC: no longer R143.1
Changed lines of the file:
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@@
 		(body_style 1)
 		(exclude_from_sim no)
-		(in_bom yes)
+		(in_bom no)
 		(on_board yes)
 		(in_pos_files yes)
@@
 			)
 		)
-		(property "Value" "10k"
+		(property "Value" "100k"
 			(at 64.135 107.315 0)
 			(show_name no)
@@
 			)
 		)
-		(property "Value" "+3V3_RTC"
+		(property "Value" "+3V3_M"
 			(at 197.485 118.745 0)
 			(show_name no)
@@
 			)
 		)
-		(property "Value" "10k"
+		(property "Value" "100k"
 			(at 209.55 130.175 0)
 			(show_name no)
